File: Kit-Brainboard.kicad_pcb (KiCad board)
At the start: 4 copper layers, 39.9 x 62.2 mm, 138 parts, among them J1 Pins_02x04_RightAngle_P2.54mm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, J2 Pins_02x05_P1.27mm_SMT, J3 USB_B_Micro_10118194-0011LF, J4 Conn_02x50, J6 Conn_02x50, Q1 MMBT3904, U13 NCP51460SN33, U14 DDR3L-RAM-4Gb_MT41K256M16TW, U15 AP6230xZ6, U16 AP6230xZ6, U17 AP6230xZ6, U18 TAR5S33, U19 TAR5S33, U2 STM32MP15xxAD, U20 AP2411SN, U3 USBLC6-2SC6, U5 NORFLASH_W25Q128JV, X1 24MHz_8pF_2x1.6mm

Commit message: WIP routing v0.1
Parts:
- C12: moved to B.Cu
- J4, J6: value Conn_02x50 -> Conn_02x40_Odd_Even; footprint mp153-devboard:Connector-100pin-P0.4mm-W3.0mm -> mp153-devboard:Connector-80pin-P0.4mm-W3.0mm
- moved D23 63.5 mm to (215.1, 45.5)
- moved D22 63.2 mm to (169.4, 92.1)
- moved D20 55.1 mm to (170.5, 96.6)
- moved D18 49.2 mm to (220.1, 45.2)
- moved D25 38.2 mm to (169.8, 107.4)
- moved D12 38.0 mm to (209.2, 117.0)
- moved D13 38.0 mm to (209.2, 121.3)
- moved D14 38.0 mm to (209.2, 125.7)
- moved D16 38.0 mm to (204.7, 117.0)
- moved D17 38.0 mm to (204.7, 121.3)
- moved D19 38.0 mm to (204.7, 125.7)
- moved D2 38.0 mm to (218.3, 117.0)
- moved D3 38.0 mm to (218.3, 121.3)
- moved D7 38.0 mm to (218.3, 125.7)
- moved D10 38.0 mm to (213.8, 125.7)
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Connections:
- J4 pad 1: /D0 -> /D28
- J4 pad 10: unconnected-(J4-Pin_10-Pad10) -> /D2
- J4 pad 11: /D13 -> /I2C2_SCL
- J4 pad 12: unconnected-(J4-Pin_12-Pad12) -> /I2C2_SCL
- J4 pad 13: /I2C2_SDA -> /D13
- J4 pad 14: unconnected-(J4-Pin_14-Pad14) -> /D13
- J4 pad 15: /D20 -> /I2C2_SDA
- J4 pad 16: unconnected-(J4-Pin_16-Pad16) -> /I2C2_SDA
- J4 pad 17: /D1 -> /D20
- J4 pad 18: unconnected-(J4-Pin_18-Pad18) -> /D20
- J4 pad 19: unconnected-(J4-Pin_19-Pad19) -> /D1
- J4 pad 2: unconnected-(J4-Pin_2-Pad2) -> /D28
- J4 pad 20: unconnected-(J4-Pin_20-Pad20) -> /D1
- J4 pad 21: unconnected-(J4-Pin_21-Pad21) -> GND
- J4 pad 22: unconnected-(J4-Pin_22-Pad22) -> GND
- J4 pad 23: unconnected-(J4-Pin_23-Pad23) -> GND
- J4 pad 24: unconnected-(J4-Pin_24-Pad24) -> GND
- J4 pad 25: /ADC-IN8 -> GNDADC
- J4 pad 26: unconnected-(J4-Pin_26-Pad26) -> GNDADC
- J4 pad 27: /D7 -> VREF+
- J4 pad 28: unconnected-(J4-Pin_28-Pad28) -> VREF+
- J4 pad 29: unconnected-(J4-Pin_29-Pad29) -> /ADC-16
- J4 pad 3: /D3 -> /D0
- J4 pad 30: unconnected-(J4-Pin_30-Pad30) -> /ADC-16
- J4 pad 31: unconnected-(J4-Pin_31-Pad31) -> /ADC-15
- J4 pad 32: unconnected-(J4-Pin_32-Pad32) -> /ADC-15
- J4 pad 33: unconnected-(J4-Pin_33-Pad33) -> /ADC-13
- J4 pad 34: unconnected-(J4-Pin_34-Pad34) -> /ADC-13
- J4 pad 35: unconnected-(J4-Pin_35-Pad35) -> /ADC-12
- J4 pad 36: unconnected-(J4-Pin_36-Pad36) -> /ADC-12
- J4 pad 37: unconnected-(J4-Pin_37-Pad37) -> /ADC-11
- J4 pad 38: unconnected-(J4-Pin_38-Pad38) -> /ADC-11
- J4 pad 39: unconnected-(J4-Pin_39-Pad39) -> /ADC-17
- J4 pad 4: unconnected-(J4-Pin_4-Pad4) -> /D0
- J4 pad 40: unconnected-(J4-Pin_40-Pad40) -> /ADC-17
- J4 pad 41: unconnected-(J4-Pin_41-Pad41) -> /ADC-9
- J4 pad 42: unconnected-(J4-Pin_42-Pad42) -> /ADC-9
- J4 pad 43: unconnected-(J4-Pin_43-Pad43) -> /ADC-14
- J4 pad 44: unconnected-(J4-Pin_44-Pad44) -> /ADC-14
- J4 pad 45: unconnected-(J4-Pin_45-Pad45) -> /ADC-5
- J4 pad 46: unconnected-(J4-Pin_46-Pad46) -> /ADC-5
- J4 pad 47: unconnected-(J4-Pin_47-Pad47) -> /ADC-8
- J4 pad 48: unconnected-(J4-Pin_48-Pad48) -> /ADC-8
- J4 pad 49: unconnected-(J4-Pin_49-Pad49) -> /ADC-4
- J4 pad 5: /D15 -> /D3
- J4 pad 50: unconnected-(J4-Pin_50-Pad50) -> /ADC-4
- J4 pad 51: unconnected-(J4-Pin_51-Pad51) -> /ADC-10
- J4 pad 52: unconnected-(J4-Pin_52-Pad52) -> /ADC-10
- J4 pad 53: unconnected-(J4-Pin_53-Pad53) -> /ADC-7
- J4 pad 54: unconnected-(J4-Pin_54-Pad54) -> /ADC-7
- J4 pad 55: unconnected-(J4-Pin_55-Pad55) -> /ADC-19_DAC1
- J4 pad 56: unconnected-(J4-Pin_56-Pad56) -> /ADC-19_DAC1
- J4 pad 57: unconnected-(J4-Pin_57-Pad57) -> /ADC-3
- J4 pad 58: unconnected-(J4-Pin_58-Pad58) -> /ADC-3
- J4 pad 59: unconnected-(J4-Pin_59-Pad59) -> /ADC-18_DAC0
- J4 pad 6: unconnected-(J4-Pin_6-Pad6) -> /D3
- J4 pad 60: unconnected-(J4-Pin_60-Pad60) -> /ADC-18_DAC0
- J4 pad 61: unconnected-(J4-Pin_61-Pad61) -> /ADC-2
- J4 pad 62: unconnected-(J4-Pin_62-Pad62) -> /ADC-2
- J4 pad 63: unconnected-(J4-Pin_63-Pad63) -> VREF+
- J4 pad 64: unconnected-(J4-Pin_64-Pad64) -> VREF+
- J4 pad 65: unconnected-(J4-Pin_65-Pad65) -> GNDADC
- J4 pad 66: unconnected-(J4-Pin_66-Pad66) -> GNDADC
- J4 pad 67: unconnected-(J4-Pin_67-Pad67) -> GND
- J4 pad 68: unconnected-(J4-Pin_68-Pad68) -> GND
- J4 pad 69: unconnected-(J4-Pin_69-Pad69) -> /D29
- J4 pad 7: /D2 -> /D15
- J4 pad 70: unconnected-(J4-Pin_70-Pad70) -> /D29
- J4 pad 71: unconnected-(J4-Pin_71-Pad71) -> /D27
- J4 pad 72: unconnected-(J4-Pin_72-Pad72) -> /D27
- J4 pad 73: unconnected-(J4-Pin_73-Pad73) -> /D26
- J4 pad 74: unconnected-(J4-Pin_74-Pad74) -> /D26
- J4 pad 75: unconnected-(J4-Pin_75-Pad75) -> /D30
- J4 pad 76: unconnected-(J4-Pin_76-Pad76) -> /D30
- J4 pad 77: unconnected-(J4-Pin_77-Pad77) -> GND
- J4 pad 78: unconnected-(J4-Pin_78-Pad78) -> GND
- J4 pad 79: unconnected-(J4-Pin_79-Pad79) -> GND
- J4 pad 8: unconnected-(J4-Pin_8-Pad8) -> /D15
- J4 pad 80: unconnected-(J4-Pin_80-Pad80) -> GND
- J4 pad 9: /I2C2_SCL -> /D2
- J6 pad 1: unconnected-(J6-Pin_1-Pad1) -> /D23
- J6 pad 10: /D18 -> /D16
- J6 pad 11: /D19 -> /D17
- J6 pad 12: /D19 -> /D17
- J6 pad 13: /D4 -> /D18
- J6 pad 14: /D4 -> /D18
- J6 pad 15: /D9 -> /D19
- J6 pad 16: /D9 -> /D19
- J6 pad 17: unconnected-(J6-Pin_17-Pad17) -> /D4
- J6 pad 18: unconnected-(J6-Pin_18-Pad18) -> /D4
- J6 pad 19: unconnected-(J6-Pin_19-Pad19) -> /D9
- J6 pad 2: /D10 -> /D23
- J6 pad 20: unconnected-(J6-Pin_20-Pad20) -> /D9
- J6 pad 21: unconnected-(J6-Pin_21-Pad21) -> Net-(J6-Pin_21)
- J6 pad 22: /SAI_SD_A -> Net-(J6-Pin_21)
- J6 pad 23: unconnected-(J6-Pin_23-Pad23) -> Net-(J6-Pin_23)
- J6 pad 24: /SAI_SD_B -> Net-(J6-Pin_23)
- J6 pad 25: unconnected-(J6-Pin_25-Pad25) -> Net-(J6-Pin_25)
- J6 pad 26: /SAI_SCK -> Net-(J6-Pin_25)
- J6 pad 27: unconnected-(J6-Pin_27-Pad27) -> +5V
- J6 pad 28: /SAI_MCLK -> +5V
- J6 pad 29: unconnected-(J6-Pin_29-Pad29) -> +5V
- J6 pad 3: unconnected-(J6-Pin_3-Pad3) -> /D10
- J6 pad 30: /SAI_FS -> +5V
- J6 pad 31: unconnected-(J6-Pin_31-Pad31) -> GND
- J6 pad 33: unconnected-(J6-Pin_33-Pad33) -> GND
- J6 pad 34: /USB_HS_D+ -> GND
- J6 pad 35: unconnected-(J6-Pin_35-Pad35) -> Net-(J6-Pin_35)
- J6 pad 36: /USB_HS_D- -> Net-(J6-Pin_35)
- J6 pad 37: unconnected-(J6-Pin_37-Pad37) -> Net-(J6-Pin_37)
- J6 pad 38: unconnected-(J6-Pin_38-Pad38) -> Net-(J6-Pin_37)
- J6 pad 39: +5V -> Net-(J6-Pin_39)
- J6 pad 4: /D12 -> /D10
- J6 pad 40: +5V -> Net-(J6-Pin_39)
- J6 pad 41: +5V -> Net-(J6-Pin_41)
- J6 pad 42: +5V -> Net-(J6-Pin_41)
- J6 pad 43: GND -> Net-(J6-Pin_43)
- J6 pad 44: GND -> Net-(J6-Pin_43)
- J6 pad 45: GND -> Net-(J6-Pin_45)
- J6 pad 46: GND -> Net-(J6-Pin_45)
- J6 pad 47: unconnected-(J6-Pin_47-Pad47) -> Net-(J6-Pin_47)
- J6 pad 48: unconnected-(J6-Pin_48-Pad48) -> Net-(J6-Pin_47)
- J6 pad 49: unconnected-(J6-Pin_49-Pad49) -> Net-(J6-Pin_49)
- J6 pad 5: /D16 -> /D22
- J6 pad 50: unconnected-(J6-Pin_50-Pad50) -> Net-(J6-Pin_49)
- J6 pad 51: unconnected-(J6-Pin_51-Pad51) -> Net-(J6-Pin_51)
- J6 pad 52: unconnected-(J6-Pin_52-Pad52) -> Net-(J6-Pin_51)
- J6 pad 53: unconnected-(J6-Pin_53-Pad53) -> Net-(J6-Pin_53)
- J6 pad 54: unconnected-(J6-Pin_54-Pad54) -> Net-(J6-Pin_53)
- J6 pad 55: unconnected-(J6-Pin_55-Pad55) -> /SAI_MCLK
- J6 pad 56: /D23 -> /SAI_MCLK
- J6 pad 57: unconnected-(J6-Pin_57-Pad57) -> /SAI_FS
- J6 pad 58: /D6 -> /SAI_FS
- J6 pad 59: unconnected-(J6-Pin_59-Pad59) -> /SAI_SCK
- J6 pad 6: /D16 -> /D22
- J6 pad 60: /D5 -> /SAI_SCK
- J6 pad 61: unconnected-(J6-Pin_61-Pad61) -> /SAI_SD_A
- J6 pad 62: /D22 -> /SAI_SD_A
- J6 pad 63: unconnected-(J6-Pin_63-Pad63) -> /SAI_SD_B
- J6 pad 64: /D21 -> /SAI_SD_B
- J6 pad 65: unconnected-(J6-Pin_65-Pad65) -> /D6
- J6 pad 66: unconnected-(J6-Pin_66-Pad66) -> /D6
- J6 pad 67: unconnected-(J6-Pin_67-Pad67) -> /D24
- J6 pad 68: unconnected-(J6-Pin_68-Pad68) -> /D24
- J6 pad 69: unconnected-(J6-Pin_69-Pad69) -> /D21
- J6 pad 7: /D17 -> /D12
- J6 pad 70: unconnected-(J6-Pin_70-Pad70) -> /D21
- J6 pad 71: unconnected-(J6-Pin_71-Pad71) -> /D5
- J6 pad 72: unconnected-(J6-Pin_72-Pad72) -> /D5
- J6 pad 73: unconnected-(J6-Pin_73-Pad73) -> GND
- J6 pad 74: unconnected-(J6-Pin_74-Pad74) -> GND
- J6 pad 75: unconnected-(J6-Pin_75-Pad75) -> /USB_HS_D+
- J6 pad 76: unconnected-(J6-Pin_76-Pad76) -> /USB_HS_D+
- J6 pad 77: unconnected-(J6-Pin_77-Pad77) -> /USB_HS_D-
- J6 pad 78: unconnected-(J6-Pin_78-Pad78) -> /USB_HS_D-
- J6 pad 79: unconnected-(J6-Pin_79-Pad79) -> GND
- J6 pad 8: /D17 -> /D12
- J6 pad 80: unconnected-(J6-Pin_80-Pad80) -> GND
- J6 pad 9: /D18 -> /D16
- U2 pad 1A3: /DEBUG2 -> /D28
- U2 pad 1H1: /ADC-IN1_DAC-OUT1 -> /ADC-19_DAC1
- U2 pad 1J1: /ADC-IN0_DAC-OUT0 -> /ADC-18_DAC0
- U2 pad 1J2: unconnected-(U2A-PB13-Pad1J2) -> /D25
- U2 pad C9: unconnected-(U2A-PB9-PadC9) -> /DEBUG2
- U2 pad N2: /ADC-IN4 -> /ADC-15
- U2 pad N3: unconnected-(U2A-PA0-PadN3) -> /ADC-16
- U2 pad P1: unconnected-(U2B-PE2-PadP1) -> /D29
- U2 pad P2: /D7 -> /ADC-12
- U2 pad P3: /ADC-IN8 -> /ADC-13
- U2 pad R3: unconnected-(U2B-PG13-PadR3) -> /D27
- U2 pad T1: /D14 -> /ADC-17
- U2 pad T2: /D8 -> /ADC-11
- U2 pad T3: /ADC-IN2 -> /ADC-14
- U2 pad U1: /D11 -> /ADC-5
- U2 pad U2: /ADC-IN6 -> /ADC-9
- U2 pad U4: /ADC-IN9 -> /ADC-10
- U2 pad V1: /ADC-IN7 -> /ADC-8
- U2 pad V12: unconnected-(U2B-PE10-PadV12) -> /D11
- U2 pad V13: unconnected-(U2A-PB2-PadV13) -> /D30
- U2 pad V2: /ADC-IN15 -> /ADC-4
- U2 pad V4: unconnected-(U2A-PB8-PadV4) -> /D26
- U2 pad W2: /ADC-IN5 -> /ADC-7
- U2 pad W3: /ADC-IN3 -> /ADC-3
- U2 pad W4: /ADC-IN14 -> /ADC-2
- U2 pad W8: unconnected-(U2B-PG9-PadW8) -> /D24
Routing:
- net /D28: track 0.00 -> 50.6 mm, vias 0 -> 2
- net /D30: track 0.00 -> 33.5 mm, vias 0 -> 2
- net /D24: track 0.00 -> 33.4 mm, vias 0 -> 2
- net /D27: track 0.00 -> 30.3 mm, vias 0 -> 2
- net /D29: track 0.00 -> 27.9 mm, vias 0 -> 2
- net /ADC-19_DAC1: track 0.00 -> 27.7 mm
- net /ADC-10: track 0.00 -> 27.4 mm, vias 0 -> 2
- net /ADC-18_DAC0: track 0.00 -> 27.2 mm
- net /D6: track 7.20 -> 33.8 mm, vias 0 -> 2
- net /ADC-16: track 0.00 -> 26.6 mm
- net GNDADC: track 69.1 -> 95.6 mm, vias 6 -> 8
- net /D26: track 0.00 -> 26.2 mm, vias 0 -> 2
- net /ADC-13: track 0.00 -> 25.9 mm
- net /ADC-14: track 0.00 -> 25.9 mm, vias 0 -> 2
- net /ADC-15: track 0.00 -> 25.6 mm
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- added copper zone on In2.Cu, net GND
- removed copper zone on In2.Cu, net (none)
- removed copper zone on In2.Cu, net +3V3
Other:
- board size 39.9 x 62.2 mm -> 39.9 x 56.4 mm
