File: Kit-Brainboard.kicad_sch (KiCad schematic)
At the start: 138 parts, among them J1 Pins_02x04_RightAngle_P2.54mm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, J2 Pins_02x05_P1.27mm_SMT, J3 USB_B_Micro_10118194-0011LF, J4 Conn_02x50, J6 Conn_02x50, Q1 MMBT3904, U13 NCP51460SN33, U14 DDR3L-RAM-4Gb_MT41K256M16TW, U15 AP6230xZ6, U16 AP6230xZ6, U17 AP6230xZ6, U18 TAR5S33, U19 TAR5S33, U2 STM32MP15xxAD, U20 AP2411SN, U3 USBLC6-2SC6, U5 NORFLASH_W25Q128JV, X1 24MHz_8pF_2x1.6mm

Commit message: WIP routing v0.1
Parts:
- removed J6: Conn_02x50, mp153-devboard:Connector-100pin-P0.4mm-W3.0mm, symbol 4ms_Connector:Conn_02x50
- added J6: Conn_02x40_Odd_Even, mp153-devboard:Connector-80pin-P0.4mm-W3.0mm, symbol Connector_Generic:Conn_02x40_Odd_Even
- J4: value Conn_02x50 -> Conn_02x40_Odd_Even; footprint mp153-devboard:Connector-100pin-P0.4mm-W3.0mm -> mp153-devboard:Connector-80pin-P0.4mm-W3.0mm; symbol 4ms_Connector:Conn_02x50 -> Connector_Generic:Conn_02x40_Odd_Even; Production Stage AB -> (none)
Connections:
- net ADC-IN14 is gone; now on net ADC-2: U2.W4 (PF11)
- net ADC-IN15 is gone; now on net ADC-4: U2.V2 (PC4)
- net +5V: now also J6.27 (Pin_27), J6.28 (Pin_28), J6.29 (Pin_29), J6.30 (Pin_30)
- net ADC-IN0_DAC-OUT0: no longer U2.1J1 (PA4)
- net ADC-IN1_DAC-OUT1: no longer U2.1H1 (PA5)
- net ADC-IN2: no longer U2.T3 (PA2)
- net ADC-IN3: no longer U2.W3 (PA6)
- net ADC-IN4: no longer U2.N2 (PA3)
- net ADC-IN5: no longer U2.W2 (PA7)
- net ADC-IN6: no longer U2.U2 (PB0)
- net ADC-IN7: no longer U2.V1 (PC5)
- net ADC-IN8: no longer J4.25 (Pin_25), U2.P3 (PC3)
- net ADC-IN9: no longer U2.U4 (PC0)
- net D0: now also J4.3 (Pin_3), J4.4 (Pin_4); no longer J4.1 (Pin_1)
- net D1: now also J4.19 (Pin_19), J4.20 (Pin_20); no longer J4.17 (Pin_17)
- net D10: now also J6.3 (Pin_3), J6.4 (Pin_4)
- net D11: now also U2.V12 (PE10); no longer U2.U1 (PB1)
- net D12: now also J6.7 (Pin_7), J6.8 (Pin_8)
- net D13: now also J4.13 (Pin_13), J4.14 (Pin_14); no longer J4.11 (Pin_11)
- net D14: no longer U2.T1 (PA1)
- net D15: now also J4.7 (Pin_7), J4.8 (Pin_8); no longer J4.5 (Pin_5)
- net D16: now also J6.10 (Pin_10), J6.9 (Pin_9)
- net D17: now also J6.11 (Pin_11), J6.12 (Pin_12)
- net D18: now also J6.13 (Pin_13), J6.14 (Pin_14)
- net D19: now also J6.15 (Pin_15), J6.16 (Pin_16)
- net D2: now also J4.10 (Pin_10), J4.9 (Pin_9); no longer J4.7 (Pin_7)
- net D20: now also J4.17 (Pin_17), J4.18 (Pin_18); no longer J4.15 (Pin_15)
- net D21: now also J6.69 (Pin_69), J6.70 (Pin_70)
- net D22: now also J6.5 (Pin_5), J6.6 (Pin_6)
- net D23: now also J6.1 (Pin_1), J6.2 (Pin_2)
- net D3: now also J4.5 (Pin_5), J4.6 (Pin_6); no longer J4.3 (Pin_3)
- net D4: now also J6.17 (Pin_17), J6.18 (Pin_18)
- net D5: now also J6.71 (Pin_71), J6.72 (Pin_72)
- net D6: now also J6.65 (Pin_65), J6.66 (Pin_66)
- net D7: no longer J4.27 (Pin_27), U2.P2 (PC2)
- net D8: no longer U2.T2 (PC1)
- net D9: now also J6.19 (Pin_19), J6.20 (Pin_20)
- net DEBUG2: now also U2.C9 (PB9); no longer U2.1A3 (PE3)
- net GND: now also J4.21 (Pin_21), J4.22 (Pin_22), J4.23 (Pin_23), J4.24 (Pin_24), J4.67 (Pin_67), J4.68 (Pin_68), J4.77 (Pin_77), J4.78 (Pin_78), J4.79 (Pin_79), J4.80 (Pin_80), J6.31 (Pin_31), J6.32 (Pin_32), J6.33 (Pin_33), J6.34 (Pin_34), J6.73 (Pin_73), J6.74 (Pin_74), J6.79 (Pin_79), J6.80 (Pin_80); no longer J4.91 (Pin_91)
- net GNDADC: now also J4.25 (Pin_25), J4.26 (Pin_26), J4.65 (Pin_65), J4.66 (Pin_66)
- net I2C2_SCL: now also J4.11 (Pin_11), J4.12 (Pin_12); no longer J4.9 (Pin_9)
- net I2C2_SDA: now also J4.15 (Pin_15), J4.16 (Pin_16); no longer J4.13 (Pin_13)
- net SAI_FS: now also J6.57 (Pin_57), J6.58 (Pin_58)
- net SAI_MCLK: now also J6.55 (Pin_55), J6.56 (Pin_56)
- net SAI_SCK: now also J6.59 (Pin_59), J6.60 (Pin_60)
- net SAI_SD_A: now also J6.61 (Pin_61), J6.62 (Pin_62)
- net SAI_SD_B: now also J6.63 (Pin_63), J6.64 (Pin_64)
- net USB_HS_D+: now also J6.75 (Pin_75), J6.76 (Pin_76)
- net USB_HS_D-: now also J6.77 (Pin_77), J6.78 (Pin_78)
- net VREF+: now also J4.27 (Pin_27), J4.28 (Pin_28), J4.63 (Pin_63), J4.64 (Pin_64)
- net D28: now reaches J4.2 (Pin_2)
- net D28: now also J4.1 (Pin_1), U2.1A3 (PE3)
- net ADC-16: now reaches J4.29 (Pin_29)
- net ADC-16: now also J4.30 (Pin_30), U2.N3 (PA0)
- net ADC-15: now reaches J4.31 (Pin_31)
- net ADC-15: now also J4.32 (Pin_32), U2.N2 (PA3)
- net ADC-13: now reaches J4.33 (Pin_33)
- net ADC-13: now also J4.34 (Pin_34), U2.P3 (PC3)
- net ADC-12: now reaches J4.35 (Pin_35)
- net ADC-12: now also J4.36 (Pin_36), U2.P2 (PC2)
- net ADC-11: now reaches J4.37 (Pin_37)
- net ADC-11: now also J4.38 (Pin_38), U2.T2 (PC1)
- net ADC-17: now reaches J4.39 (Pin_39)
- net ADC-17: now also J4.40 (Pin_40), U2.T1 (PA1)
- net ADC-9: now reaches J4.41 (Pin_41)
- net ADC-9: now also J4.42 (Pin_42), U2.U2 (PB0)
- net ADC-14: now reaches J4.43 (Pin_43)
- net ADC-14: now also J4.44 (Pin_44), U2.T3 (PA2)
- net ADC-5: now reaches J4.45 (Pin_45)
- net ADC-5: now also J4.46 (Pin_46), U2.U1 (PB1)
- net ADC-8: now reaches J4.47 (Pin_47)
- net ADC-8: now also J4.48 (Pin_48), U2.V1 (PC5)
- net ADC-4: now reaches J4.49 (Pin_49)
- net ADC-4: now also J4.50 (Pin_50)
- net ADC-10: now reaches J4.51 (Pin_51)
- net ADC-10: now also J4.52 (Pin_52), U2.U4 (PC0)
- net ADC-7: now reaches J4.53 (Pin_53)
- net ADC-7: now also J4.54 (Pin_54), U2.W2 (PA7)
- net ADC-19_DAC1: now reaches J4.55 (Pin_55)
- net ADC-19_DAC1: now also J4.56 (Pin_56), U2.1H1 (PA5)
- net ADC-3: now reaches J4.57 (Pin_57)
- net ADC-3: now also J4.58 (Pin_58), U2.W3 (PA6)
- net ADC-18_DAC0: now reaches J4.59 (Pin_59)
- net ADC-18_DAC0: now also J4.60 (Pin_60), U2.1J1 (PA4)
- net ADC-2: now reaches J4.61 (Pin_61)
- net ADC-2: now also J4.62 (Pin_62)
- net D29: now reaches J4.69 (Pin_69)
- net D29: now also J4.70 (Pin_70), U2.P1 (PE2)
- net D27: now reaches J4.71 (Pin_71)
- net D27: now also J4.72 (Pin_72), U2.R3 (PG13)
- net D26: now reaches J4.73 (Pin_73)
- net D26: now also J4.74 (Pin_74), U2.V4 (PB8)
- net D30: now reaches J4.75 (Pin_75)
- net D30: now also J4.76 (Pin_76), U2.V13 (PB2)
- net D25: now reaches U2.1J2 (PB13)
- net D24: now reaches U2.W8 (PG9)
- net D24: now also J6.67 (Pin_67), J6.68 (Pin_68)
- new net: J6.21 (Pin_21), J6.22 (Pin_22)
- new net: J6.23 (Pin_23), J6.24 (Pin_24)
- new net: J6.25 (Pin_25), J6.26 (Pin_26)
- new net: J6.35 (Pin_35), J6.36 (Pin_36)
- new net: J6.37 (Pin_37), J6.38 (Pin_38)
- new net: J6.39 (Pin_39), J6.40 (Pin_40)
- new net: J6.41 (Pin_41), J6.42 (Pin_42)
- new net: J6.43 (Pin_43), J6.44 (Pin_44)
- new net: J6.45 (Pin_45), J6.46 (Pin_46)
- new net: J6.47 (Pin_47), J6.48 (Pin_48)
- new net: J6.49 (Pin_49), J6.50 (Pin_50)
- new net: J6.51 (Pin_51), J6.52 (Pin_52)
- new net: J6.53 (Pin_53), J6.54 (Pin_54)
- no-connect marks 68 -> 59
Other:
- note added: "Changed: DEBUG2 Rename CODEC_RESET to D20 (PE12) ??? Add up to D30 Add up to ADC-IN16 D8=>ADC, D14=>ADC, D7 is missing"
- note added: "D11"
- note added: "D14"
- note added: "D7"
- note added: "D8"
- note added: "I2C1_SCL"
- note added: "I2C1_SDA"
- note added: "SAI1_FS_A"
- note added: "SAI1_MCLK"
- note added: "SAI1_SCK_A"
- note added: "SAI1_SD_A"
- note added: "SAI1_SD_B"
- note added: "SAI4_SCK_A"
- note added: "SAI4_SD_B"
- note removed: "ADC-IN10"
- note removed: "ADC-IN11"
- note removed: "ADC-IN12"
- note removed: "ADC-IN13"
- note removed: "Changed: DEBUG2 => PE3 Rename CODEC_RESET to D20 (PE12) ??? Add ADC-IN14 (PF11, ADC1_INP2) Add ADC-IN15 (PC4, ADC1_INP4)"
- note removed: "TODO: I2C on top header More GPIOs All ADCs"
