File: mp153-devboard.kicad_pcb (KiCad board)
At the start: 4 copper layers, 39.9 x 56.4 mm, 138 parts, among them J1 Pins_02x04_RightAngle_P2.54mm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, J2 Pins_02x05_P1.27mm_SMT, J3 USB_B_Micro_10118194-0011LF, J4 Conn_02x40_Odd_Even, J6 Conn_02x40_Odd_Even, Q1 MMBT3904, U13 NCP51460SN33, U14 DDR3L-RAM-4Gb_MT41K256M16TW, U15 AP6230xZ6, U16 AP6230xZ6, U17 AP6230xZ6, U18 TAR5S33, U19 TAR5S33, U2 STM32MP15xxAD, U20 AP2411SN, U3 USBLC6-2SC6, U5 NORFLASH_W25Q128JV, X1 24MHz_8pF_2x1.6mm

Commit message: Finish v0.1 dev board
Parts:
- removed D1, D10, D12, D13, D14, D15, D16, D17, D18, D19, D2, D20, D21, D22, D23, D24, D25, D26, D3, D4, D5, D6, D7, D8, D9: BAT54S, 4ms_Package_SOT:SOT23-3_PO132
- added H1: Spacer Nylon, fits 3mm hole, 4ms_Hardware:MountingHole_Generic_3mm, F.Cu at (226.6, 52.6)
- added H2: Spacer Nylon, fits 3mm hole, 4ms_Hardware:MountingHole_Generic_3mm, F.Cu at (192.6, 52.6)
- added H3: Spacer Nylon, fits 3mm hole, 4ms_Hardware:MountingHole_Generic_3mm, F.Cu at (192.6, 102.6)
- added H4: Spacer Nylon, fits 3mm hole, 4ms_Hardware:MountingHole_Generic_3mm, F.Cu at (226.6, 102.6)
- J1, J2: moved to B.Cu
- J4, J6: value Conn_02x40_Odd_Even -> Pins_02x40_P0.4mm_W3.0mm_SMT
- moved S2 30.4 mm to (193.9, 64.4)
- moved JP1 7.14 mm to (196.4, 88.3)
- moved J2 5.75 mm to (193.7, 92.7)
- moved R74 4.91 mm to (200.8, 91.8), turned to -90 degrees
- moved C67 1.39 mm to (195.7, 72.3)
- moved J1 0.59 mm to (192.1, 75.8)
- moved R61 0.36 mm to (195.3, 69.7)
Connections:
- J4 pad 15: /I2C2_SDA -> /D8
- J4 pad 16: /I2C2_SDA -> /D8
- J4 pad 17: /D20 -> /I2C2_SDA
- J4 pad 18: /D20 -> /I2C2_SDA
- J4 pad 19: /D1 -> /D20
- J4 pad 20: /D1 -> /D20
- J4 pad 21: GND -> /D1
- J4 pad 22: GND -> /D1
- J6 pad 10: /D16 -> /D17
- J6 pad 11: /D17 -> /D12
- J6 pad 12: /D17 -> /D12
- J6 pad 21: Net-(J6-Pin_21) -> GND
- J6 pad 22: Net-(J6-Pin_21) -> GND
- J6 pad 23: Net-(J6-Pin_23) -> +5V
- J6 pad 24: Net-(J6-Pin_23) -> +5V
- J6 pad 25: Net-(J6-Pin_25) -> +5V
- J6 pad 26: Net-(J6-Pin_25) -> +5V
- J6 pad 35: Net-(J6-Pin_35) -> GND
- J6 pad 36: Net-(J6-Pin_35) -> GND
- J6 pad 37: Net-(J6-Pin_37) -> GND
- J6 pad 38: Net-(J6-Pin_37) -> GND
- J6 pad 39: Net-(J6-Pin_39) -> GND
- J6 pad 40: Net-(J6-Pin_39) -> GND
- J6 pad 41: Net-(J6-Pin_41) -> /D7
- J6 pad 42: Net-(J6-Pin_41) -> /D7
- J6 pad 43: Net-(J6-Pin_43) -> /SAI_MCLK
- J6 pad 44: Net-(J6-Pin_43) -> /SAI_MCLK
- J6 pad 45: Net-(J6-Pin_45) -> /SAI_FS
- J6 pad 46: Net-(J6-Pin_45) -> /SAI_FS
- J6 pad 47: Net-(J6-Pin_47) -> /SAI_SCK
- J6 pad 48: Net-(J6-Pin_47) -> /SAI_SCK
- J6 pad 49: Net-(J6-Pin_49) -> /SAI_SD_A
- J6 pad 50: Net-(J6-Pin_49) -> /SAI_SD_A
- J6 pad 51: Net-(J6-Pin_51) -> /SAI_SD_B
- J6 pad 52: Net-(J6-Pin_51) -> /SAI_SD_B
- J6 pad 53: Net-(J6-Pin_53) -> GND
- J6 pad 54: Net-(J6-Pin_53) -> GND
- J6 pad 55: /SAI_MCLK -> /D6
- J6 pad 56: /SAI_MCLK -> /D6
- J6 pad 57: /SAI_FS -> /D24
- J6 pad 58: /SAI_FS -> /D24
- J6 pad 59: /SAI_SCK -> /D21
- J6 pad 60: /SAI_SCK -> /D21
- J6 pad 61: /SAI_SD_A -> /D5
- J6 pad 62: /SAI_SD_A -> /D5
- J6 pad 63: /SAI_SD_B -> /D11
- J6 pad 64: /SAI_SD_B -> /D11
- J6 pad 65: /D6 -> +3V3
- J6 pad 66: /D6 -> +3V3
- J6 pad 67: /D24 -> +3V3
- J6 pad 68: /D24 -> +3V3
- J6 pad 69: /D21 -> GND
- J6 pad 7: /D12 -> /D16
- J6 pad 70: /D21 -> GND
- J6 pad 71: /D5 -> /USB_VBUS_JACK
- J6 pad 72: /D5 -> /USB_VBUS_JACK
- J6 pad 75: /USB_HS_D+ -> /USB_HS_D-
- J6 pad 76: /USB_HS_D+ -> /USB_HS_D-
- J6 pad 77: /USB_HS_D- -> /USB_HS_D+
- J6 pad 78: /USB_HS_D- -> /USB_HS_D+
- J6 pad 8: /D12 -> /D16
- J6 pad 9: /D16 -> /D17
- U2 pad 1J2: /D25 -> unconnected-(U2A-PB13-Pad1J2)
- U2 pad B2: unconnected-(U2B-PE6-PadB2) -> /D8
- U2 pad U16: unconnected-(U2A-PA10-PadU16) -> /D7
Routing:
- net /USB_VBUS_JACK: track 3.70 -> 47.4 mm, vias 1 -> 2
- net GND: track 215.5 -> 254.0 mm, vias 81 -> 90
- net /D11: track 1.57 -> 38.4 mm, vias 0 -> 2
- net +5V: track 121.8 -> 158.3 mm
- net /D7: track 0.00 -> 34.4 mm, vias 0 -> 2
- net +3V3: track 47.7 -> 74.0 mm
- net /NRST: track 104.6 -> 78.8 mm, vias 4 -> 3
- net /SAI_MCLK: track 34.3 -> 57.4 mm, vias 2 -> 4
- net /D8: track 0.00 -> 21.5 mm
- net GNDADC: track 95.6 -> 75.5 mm, vias 8 -> 6
- net /D9: track 27.1 -> 42.5 mm
- net /D4: track 27.6 -> 42.4 mm
- net /D19: track 26.9 -> 41.5 mm
- net /JTCK_SWCLK: track 16.2 -> 30.8 mm, vias 2 -> 3
- net /D10: track 28.9 -> 43.3 mm
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Other:
- outline, holes or cut-outs redrawn
- board text added: "1"
- board text added: "2"
- board text added: "79"
- board text added: "80"
- board text added: "MP153 Devboard v0.1"
- board text removed: "Brainboard MP15x p5"
