File: mp153-devboard.kicad_sch (KiCad schematic)
At the start: 138 parts, among them J1 Pins_02x04_RightAngle_P2.54mm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, J2 Pins_02x05_P1.27mm_SMT, J3 USB_B_Micro_10118194-0011LF, J4 Conn_02x40_Odd_Even, J6 Conn_02x40_Odd_Even, Q1 MMBT3904, U13 NCP51460SN33, U14 DDR3L-RAM-4Gb_MT41K256M16TW, U15 AP6230xZ6, U16 AP6230xZ6, U17 AP6230xZ6, U18 TAR5S33, U19 TAR5S33, U2 STM32MP15xxAD, U20 AP2411SN, U3 USBLC6-2SC6, U5 NORFLASH_W25Q128JV, X1 24MHz_8pF_2x1.6mm

Commit message: Finish v0.1 dev board
Parts:
- removed D1, D10, D12, D13, D14, D15, D16, D17, D18, D19, D2, D20, D21, D22, D23, D24, D25, D26, D3, D4, D5, D6, D7, D8, D9: BAT54S, 4ms_Package_SOT:SOT23-3_PO132, symbol 4ms_Diode:BAT54S
- added H1, H2, H3, H4: Spacer Nylon, fits 3mm hole, 4ms_Hardware:MountingHole_Generic_3mm, symbol 4ms_Hardware:Spacer Nylon, Unthreaded, Height=11mm, ID {gt}= 3mm, OD {lt} 6mm
- J2: JLCPCB ID (none) -> C598540
- J3: JLCPCB ID (none) -> C5407473
- J4, J6: value Conn_02x40_Odd_Even -> Pins_02x40_P0.4mm_W3.0mm_SMT; symbol Connector_Generic:Conn_02x40_Odd_Even -> 4ms_Connector:Pins_02x40_P0.4mm_W3.0mm_SMT; Alt Part Number (none) -> DF40HC(3.0)-80DP-0.4V(51); JLCPCB ID (none) -> C294544; Manufacturer (none) -> Hirose; Part Number (none) -> DF40C-80DP-0.4V(51)
- S1, S2, S3: Alt JLCPCB ID (none) -> C2689538; JLCPCB ID (none) -> C2689521; Manufacturer 2 (none) -> C&K Switches; Part Number 2 (none) -> PTS526 SK15 SMTR2 LFS; Specifications (none) -> Tact button, NO,
- U15, U16, U17: JLCPCB ID (none) -> C1880992
Connections:
- net +3V3: now also J6.65 (Pin_65), J6.66 (Pin_66), J6.67 (Pin_67), J6.68 (Pin_68)
- net +5V: now also J6.23 (Pin_23), J6.24 (Pin_24), J6.25 (Pin_25), J6.26 (Pin_26)
- net D1: now also J4.21 (Pin_21), J4.22 (Pin_22); no longer J4.19 (Pin_19), J4.20 (Pin_20)
- net D11: now also J6.63 (Pin_63), J6.64 (Pin_64)
- net D12: now also J6.11 (Pin_11), J6.12 (Pin_12); no longer J6.7 (Pin_7), J6.8 (Pin_8)
- net D16: now also J6.7 (Pin_7), J6.8 (Pin_8); no longer J6.10 (Pin_10), J6.9 (Pin_9)
- net D17: now also J6.10 (Pin_10), J6.9 (Pin_9); no longer J6.11 (Pin_11), J6.12 (Pin_12)
- net D20: now also J4.19 (Pin_19), J4.20 (Pin_20); no longer J4.17 (Pin_17), J4.18 (Pin_18)
- net D21: now also J6.59 (Pin_59), J6.60 (Pin_60); no longer J6.69 (Pin_69), J6.70 (Pin_70)
- net D24: now also J6.57 (Pin_57), J6.58 (Pin_58); no longer J6.67 (Pin_67), J6.68 (Pin_68)
- net D5: now also J6.61 (Pin_61), J6.62 (Pin_62); no longer J6.71 (Pin_71), J6.72 (Pin_72)
- net D6: now also J6.55 (Pin_55), J6.56 (Pin_56); no longer J6.65 (Pin_65), J6.66 (Pin_66)
- net D7: now also J6.41 (Pin_41), J6.42 (Pin_42), U2.U16 (PA10)
- net D8: now also J4.15 (Pin_15), J4.16 (Pin_16), U2.B2 (PE6)
- net GND: now also J6.21 (Pin_21), J6.22 (Pin_22), J6.35 (Pin_35), J6.36 (Pin_36), J6.37 (Pin_37), J6.38 (Pin_38), J6.39 (Pin_39), J6.40 (Pin_40), J6.53 (Pin_53), J6.54 (Pin_54), J6.69 (Pin_69), J6.70 (Pin_70); no longer J4.21 (Pin_21), J4.22 (Pin_22)
- net I2C2_SDA: now also J4.17 (Pin_17), J4.18 (Pin_18); no longer J4.15 (Pin_15), J4.16 (Pin_16)
- net SAI_FS: now also J6.45 (Pin_45), J6.46 (Pin_46); no longer J6.57 (Pin_57), J6.58 (Pin_58)
- net SAI_MCLK: now also J6.43 (Pin_43), J6.44 (Pin_44); no longer J6.55 (Pin_55), J6.56 (Pin_56)
- net SAI_SCK: now also J6.47 (Pin_47), J6.48 (Pin_48); no longer J6.59 (Pin_59), J6.60 (Pin_60)
- net SAI_SD_A: now also J6.49 (Pin_49), J6.50 (Pin_50); no longer J6.61 (Pin_61), J6.62 (Pin_62)
- net SAI_SD_B: now also J6.51 (Pin_51), J6.52 (Pin_52); no longer J6.63 (Pin_63), J6.64 (Pin_64)
- net USB_HS_D+: now also J6.77 (Pin_77), J6.78 (Pin_78); no longer J6.75 (Pin_75), J6.76 (Pin_76)
- net USB_HS_D-: now also J6.75 (Pin_75), J6.76 (Pin_76); no longer J6.77 (Pin_77), J6.78 (Pin_78)
- net USB_VBUS_JACK: now also J6.71 (Pin_71), J6.72 (Pin_72)
- net D25: no longer names the net of U2.1J2 (PB13)
Other:
- note added: "3.3V for peripherals Rank 2 Brainboard uses 140mA max/typ (est 43mA of 12V)"
- note added: "Carrier board can use 3.3V max 500mA(??)"
- note added: "Carrier board must supply +5V here"
- note added: "Carrier board should use VREF and GNDADC for all ADC circuitry"
- note added: "Debugging"
- note added: "NORTH"
- note added: "PROCESSOR"
- note added: "SOUTH"
- note added: "SPI3_MISO"
- note added: "SPI3_MOSI"
- note added: "SPI3_NSS"
- note added: "SPI3_SCK"
- note added: "SPI4_MISO"
- note added: "SPI4_MOSI"
- note added: "SPI4_NSS"
- note added: "SPI4_SCK"
- note added: "USB"
- note removed: "3.3V for peripherals Rank 2 140mA max/typ (est 43mA of 12V)"
- note removed: "Changed: DEBUG2 Rename CODEC_RESET to D20 (PE12) ??? Add up to D30 Add up to ADC-IN16 D8=>ADC, D14=>ADC, D7 is missing"
- note removed: "D11"
- note removed: "D7"
- note removed: "D8"
- note removed: "NOTE: 8 more 0.1uF caps are required from VDD_CORE to GND"
- note removed: "PROCESSOR PORTS"
- note removed: "TIM"
- note removed: "UART4_RX"
- note removed: "UART4_TX"
- note removed: "UART5_RX"
- note removed: "UART5_TX"
- moved on the sheet: C109, C41, C44, C45, C46, C47, C48, C49, C50, C51, C52, C53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
