File: mp153-devboard.kicad_sch (KiCad schematic)
At the start: 117 parts, among them CON1 microSDCon_SMT_104031-0811, J1 Pins_02x04_RightAngle_P2.54mm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, J2 Pins_02x05_P1.27mm_SMT, J3 USB-C_Receptacle_Molex_217179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, J4 Pins_02x40_P0.4mm_W3.0mm_SMT, J5 Conn_01x02, J6 Pins_02x40_P0.4mm_W3.0mm_SMT, U13 NCP51460SN33, U14 DDR3L-RAM-4Gb_MT41K256M16TW, U15 AP6230xZ6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

Commit message: devboard v0.1: increased spacing between zones on inner layers. Vias => 0.25mm holes
Connections:
- net I2C2_SCL renamed D25
- net I2C2_SDA renamed D14
Other:
- note added: "ADC"
- note added: "Aux I2S (SAI1)"
- note added: "Carrier board must supply +5V to North header or else use USB jack with J5 jumped"
- note added: "I2C 1"
- note added: "I2C 2"
- note added: "I2C 3"
- note added: "I2C 5"
- note added: "I2C 6"
- note added: "I2C2_SCL"
- note added: "I2C2_SDA"
- note added: "Main I2S (SAI)"
- note added: "SD Card"
- note added: "SPI 2"
- note added: "SPI 3"
- note added: "SPI 4"
- note removed: "Carrier board must supply +5V here or else use USB jack with SW1 switched ON"
- moved on the sheet: CON1, J3, J4, J5, R10, R11, R4, R5, U3

Commit message: Add note to devboard schematic
Other:
- note added: "FIXES for p1 to make p2: - Should we run USB_HS_DP/DM to the mezzanine? Right now we have U3 between the uC pins and the mezzanine"
Changed lines of the file:
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@@
+		)
+	)
+	(text "FIXES for p1 to make p2:\n- Should we run USB_HS_DP/DM to the mezzanine? Right now we have U3 between the uC pins and the mezzanine"
+		(exclude_from_sim no)
+		(at 273.304 -20.32 0)
+		(effects
+			(font
+				(size 1.905 1.905)
+			)
+			(justify left)
 		)
 	)

Commit message: Schematic notes (v0.1)
Other:
- note added: "B0"
- note added: "B1"
- note added: "B2"
- note added: "B3"
- note added: "B4"
- note added: "B5"
- note added: "B6"
- note added: "CLK"
- note added: "DE"
- note added: "FIXES for p1 to make p2: - SDMMC1 pins missing 10k pull-ups - Orientation of BOOT switch is unclear (JLC placed it backwards on first run)"
- note added: "G0"
- note added: "G1"
- note added: "G2"
- note added: "G3"
- note added: "G4"
- note added: "G5"
- note added: "G6"
- note added: "HSYNC"
- note added: "HSYNC conflicts with PC6 (UART_TX) - Route PC6 to mezzanine. Maybe route PG14 (USART6_TX) to debug header, or use different UART"
- note added: "LCD_B3: route PD10 to mezzanine (replace any pin if needed)"
- note added: "LCD_G3 conflicts with DEBUG3: - Route PE11 to mezzanine header and use a different pin for DEBUG3"
- note added: "LCD_G6 conflicts with PC7 (UART_RX) - Route PC7 to mezzanine. Use PG9 for USART6_RX (or else choose diff. UART)"
- note added: "R0"
- note added: "R1"
- note added: "R2"
- note added: "R3"
- note added: "R4"
- note added: "R5"
- note added: "R6"
- note added: "SD_CARD_DETECT"
- note added: "To provide 18-bit RGB interface:"
- note added: "VSYNC"
- note removed: "FIXES for p1 to make p2: - Should we run USB_HS_DP/DM to the mezzanine? Right now we have U3 between the uC pins and the mezzanine"
- note removed: "SPI4_NSS"

Commit message: More notes on v0.1 devboard schematic. Updated cubemx file for v0.1
Other:
- note removed: "CLK"
Changed lines of the file:
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@@
-		)
-	)
-	(text "CLK"
-		(exclude_from_sim no)
-		(at 219.964 360.934 0)
-		(effects
-			(font
-				(size 1.27 1.27)
-			)
 		)
 	)
@@
 		)
 	)
-	(text "CLK"
-		(exclude_from_sim no)
-		(at 276.098 343.154 0)
-		(effects
-			(font
-				(size 1.27 1.27)
-			)
-		)
-	)

Commit message: devboard v0.1: rename all header pins
No electrical changes made: only renamed pins to use PX# style (e.g. "PA0") instead of D# style (e.g. "D23")
Connections:
- net ADC-10 renamed PC0
- net ADC-11 renamed PC1
- net ADC-12 renamed PC2
- net ADC-13 renamed PC3
- net ADC-14 renamed PA2
- net ADC-15 renamed PA3
- net ADC-16 renamed PA0
- net ADC-17 renamed PA1
- net ADC-18_DAC0 renamed PA4
- net ADC-19_DAC1 renamed PA5
- net ADC-2 renamed PF11
- net ADC-3 renamed PA6
- net ADC-4 renamed PC4
- net ADC-5 renamed PB1
- net ADC-7 renamed PA7
- net ADC-8 renamed PC5
- net ADC-9 renamed PB0
- net D0 renamed PA9
- net D1 renamed PE13
- net D10 renamed PA8
- net D11 renamed PE10
- net D12 renamed PE4
- net D13 renamed PD1
- net D14 renamed PG15
- net D15 renamed PD0
- net D16 renamed PC8
- net D17 renamed PC9
- net D18 renamed PC10
- net D19 renamed PC11
- net D2 renamed PB7
- net D20 renamed PE12
- net D21 renamed PA12
- net D22 renamed PB15
- net D23 renamed PB14
- net D24 renamed PG9
- net D25 renamed PD7
- net D26 renamed PB8
- net D27 renamed PG13
- net D28 renamed PE3
- net D29 renamed PE2
- net D3 renamed PB4
- net D30 renamed PB2
- net D4 renamed PD2
- net D5 renamed PA11
- net D6 renamed PB10
- net D7 renamed PA10
- net D8 renamed PE6
- net D9 renamed PC12
- net SAI_FS renamed PD12
- net SAI_MCLK renamed PE0
- net SAI_SCK renamed PD13
- net SAI_SD_A renamed PD11
- net SAI_SD_B renamed PG10
Other:
- note added: "A"
- note added: "ADC-10"
- note added: "ADC-11"
- note added: "ADC-12"
- note added: "ADC-13"
- note added: "ADC-14"
- note added: "ADC-15"
- note added: "ADC-16"
- note added: "ADC-17"
- note added: "ADC-18"
- note added: "ADC-18_DAC0"
- note added: "ADC-19"
- note added: "ADC-19_DAC1"
- note added: "ADC-2"
- note added: "ADC-3"
- note added: "ADC-4"
- note added: "ADC-5"
- note added: "ADC-7"
- note added: "ADC-8"
- note added: "ADC-9"
- note added: "B"
- note added: "DAC0"
- note added: "DAC1"
- note added: "SAI2_FS"
- note added: "SAI2_MCLK"
- note added: "SAI2_SCK"
- note added: "SAI2_SD_A"
- note added: "SAI2_SD_B"
- note removed: "ADC"
- note removed: "Aux I2S (SAI1)"
- note removed: "D14"
- note removed: "I2C 1"
- note removed: "I2C 2"
- note removed: "I2C 3"
- note removed: "I2C 5"
- note removed: "I2C 6"
- note removed: "Main I2S (SAI)"
- note removed: "NORTH"
- note removed: "SD Card"
- note removed: "SOUTH"
- note removed: "SPI 2"
- note removed: "SPI 3"
- note removed: "SPI 4"
