File: carrier board/mp153-carrier-board.kicad_sch (KiCad schematic)
At the start: 27 parts, among them J3 USB_B_Micro_10118194-0011LF, J4 Socket_02x40_P0.4mm_W3.0mm_SMT, J5 3.5mm_Mono_Switched_sm, J6 Socket_02x40_P0.4mm_W3.0mm_SMT, J7 Eurorack_Power_16pin_Unshroud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, J9 3.5mm_Mono_Switched_sm, U1 TL072H

Commit message: Cleanup carrier board example
Parts:
- removed J3: USB_B_Micro_10118194-0011LF, Connector_USB:USB_Micro-B_Amphenol_10118194_Horizontal, symbol 4ms_Connector:USB_B_Micro_10118194-0011LF
- added J1: USB-C_Receptacle_Molex_2171790001, 4ms_Connector:USB_C_Receptacle_Molex_2171790001, symbol 4ms_Connector:USB-C_Receptacle_Molex_2171790001
- added R3, R4: 5.1k_0603, 4ms_Resistor:R_0603, symbol 4ms_Resistor_0603:5.1k_0603
Connections:
- net GND: now also J1.A1B12 (GND1), J1.B1A12 (GND3), J1.SH1 (Shield1), J1.SH2 (Shield2), J1.SH3 (Shield3), J1.SH4 (Shield4), R3.2, R4.2
- net USB_HS_D+: now also J1.A6 (D+1), J1.B6 (D+2)
- net USB_HS_D-: now also J1.A7 (D-1), J1.B7 (D-2)
- net USB_VBUS_JACK: now also J1.A4B9 (VBUS1), J1.B4A9 (VBUS3)
- new net: J1.A5 (CC1), R4.1
- new net: J1.B5 (CC2), R3.1
- no-connect marks 5 -> 6
Other:
- note added: "USB"

Commit message: Carrier-board: Added codec and audio in/out
Parts:
- added C147, C148, C149, C150: 180pF_0402_25V, 4ms_Capacitor:C_0402, symbol 4ms_Capacitor:180pF_0402_25V
- added C152, C153: 820pF_0402_10v, 4ms_Capacitor:C_0402, symbol 4ms_Capacitor:820pF_0402_10v
- added C41: 100nF_0402_16V, 4ms_Capacitor:C_0402, symbol 4ms_Capacitor:100nF_0402_16V
- added C42, C48: 220pF_0603_25V, 4ms_Capacitor:C_0603, symbol 4ms_Capacitor:220pF_0603_25V
- added C44: 22uF_0805_10V, 4ms_Capacitor:C_0805, symbol 4ms_Capacitor:22uF_0805_10V
- added C45: 0.1uF_0603_16V, 4ms_Capacitor:C_0603, symbol 4ms_Capacitor:0.1uF_0603_16V
- added C46, C49, C52: 2.2uF_0603_25V, 4ms_Capacitor:C_0603, symbol 4ms_Capacitor:2.2uF_0603_25V
- added C51: 10uF_0603_10V, 4ms_Capacitor:C_0603, symbol 4ms_Capacitor:10uF_0603_10V
- added C71, C72, C75, C76, C77, C78: 100nF_0402_50V, 4ms_Capacitor:C_0402, symbol 4ms_Capacitor:100nF_0402_50V
- added NT1: NetTie_2, NetTie:NetTie-2_SMD_Pad0.5mm, symbol Device:NetTie_2
- added R10, R14, R158, R159, R162, R163, R6, R7: 10k_0402, 4ms_Resistor:R_0402, symbol 4ms_Resistor_0402:10k_0402
- added R152, R153, R44, R52, R54, R55: 1k_0402, 4ms_Resistor:R_0402, symbol 4ms_Resistor_0402:1k_0402
- added R157, R160, R161, R164: 24k_0402, 4ms_Resistor:R_0402, symbol 4ms_Resistor_0402:24k_0402
- added R42, R50: 14k_0402, 4ms_Resistor:R_0402, symbol 4ms_Resistor_0402:14k_0402
- added R43, R51: 100k_0402, 4ms_Resistor:R_0402, symbol 4ms_Resistor_0402:100k_0402
- added R47, R48: 4.7k_0402, 4ms_Resistor:R_0402, symbol 4ms_Resistor_0402:4.7k_0402
- added R49, R53: 1M_0402, 4ms_Resistor:R_0402, symbol 4ms_Resistor_0402:1M_0402
- added U11, U12, U8: NJM2068, 4ms_Package_SSOP:TSSOP-8_4.4x3mm_Pitch0.65mm, symbol 4ms_IC:NJM2068
- added U9: PCM3060PW, Package_SO:TSSOP-28_4.4x9.7mm_P0.65mm, symbol 4ms_IC:PCM3060PW
- added V1: AP2120N-5.0TRG1, 4ms_Package_SOT:SOT23-3_PO132, symbol 4ms_Regulator:AP2120N-5.0TRG1
- renumbered R6 to R8
Connections:
- net +12V: now also C49.1, C71.1, C75.1, C77.1, U11.8 (V+), U12.8 (V+), U8.8 (V+), V1.3 (VI)
- net +3V3: now also C41.1, R47.2, R48.2, U9.7 (VDD)
- net -12VA: now also C72.1, C76.1, C78.1, U11.4 (V-), U12.4 (V-), U8.4 (V-)
- net D10: now also R47.1, U9.1 (MC/SCL/FMT)
- net D17: now also R48.1, U9.2 (MD/SDA/DEMP)
- net D7: now also U9.15 (~{RST})
- net GND: now also C41.2, C71.2, C72.2, C75.2, C76.2, C77.2, C78.2, NT1.2, R49.2, R53.2, U9.27 (~{MS}/ADR/IFMD), U9.28 (MODE), U9.8 (DGND)
- net SAI_FS: now also U9.11 (LRCK2), U9.4 (LRCK1)
- net SAI_MCLK: now also U9.6 (SCKI1), U9.9 (SCKI2)
- net SAI_SCK: now also U9.10 (BCK2), U9.5 (BCK1)
- net SAI_SD_A: now also U9.12 (DIN)
- net SAI_SD_B: now also U9.3 (DOUT)
- new net: C153.2, R14.2, R163.2, R164.2
- new net: C147.1, R152.2, R157.1, U12.7
- new net: C152.1, R157.2, R158.2, R6.2
- new net: C48.1, R50.1, R54.2, U11.7
- new net: C48.2, R50.2, R51.1, U11.6 (-)
- new net: C150.2, R163.1, U12.3 (+)
- new net: R44.1, R49.1, U8.3 (+)
- new net: C149.1, R153.2, R161.1, U12.1
- new net: C153.1, R10.2, R161.2, R162.2
- new net: C147.2, R158.1, U12.6 (-)
- new net: C152.2, R159.2, R160.2, R7.2
- new net: C149.2, R162.1, U12.2 (-)
- new net: C42.1, R42.1, R55.2, U8.7
- new net: C42.2, R42.2, R43.1, U8.6 (-)
- new net: R52.1, R53.1, U11.3 (+)
- new net: C46.2, U8.1, U8.2 (-)
- new net: C148.2, R159.1, U12.5 (+)
- new net: C52.1, R51.2
- new net: C52.2, U11.1, U11.2 (-)
- new net: C46.1, R43.2
- new net +5VA: C51.1, U9.24 (VCC), V1.2 (VO)
- new net AUDIO_IN1: R44.2
- new net AUDIO_IN2: R52.2
- new net AUDIO_OUT1: R152.1
- new net AUDIO_OUT2: R153.1
- new net CODEC_IN_L: R55.1, U9.25 (VINL)
- new net CODEC_IN_R: R54.1, U9.26 (VINR)
- new net CODEC_OUT_L+: R7.1, U9.20 (VOUTL+)
- new net CODEC_OUT_L-: R6.1, U9.19 (VOUTL-)
- new net CODEC_OUT_R+: R14.1, U9.18 (VOUTR+)
- new net CODEC_OUT_R-: R10.1, U9.17 (VOUTR-)
- new net GNDA: C148.1, C150.1, C44.2, C45.2, C49.2, C51.2, NT1.1, R160.1, R164.1, U9.16 (SGND), U9.22 (AGND2), U9.23 (AGND1), V1.1 (GND)
- new net VCOM: C44.1, C45.1, U11.5 (+), U8.5 (+), U9.21 (VCOM)
- no-connect marks 6 -> 8
Other:
- note added: "AUDIO"
- moved on the sheet: C3, C4, C5, C6, C7, D2, D3, J7

Commit message: Finished carrier board. Produced JLC files
Parts:
- added J10, J11, J12, J13: 3.5mm_Mono_Switched_sm, 4ms_Jack:EighthInch_PJ398SM, symbol 4ms_Jack:3.5mm_Mono_Switched_sm
- added unit 2 of POT1
- C44: value 22uF_0805_10V -> 22uF_0805_25V; symbol 4ms_Capacitor:22uF_0805_10V -> 4ms_Capacitor:22uF_0805_25V; Display 22uF/10V -> 22uF/25V; Manufacturer Taiyo Yuden -> Murata; Part Number LMK212BBJ226MG-T -> GRM21BR61E226ME44L; Specifications 22uF, Min. 10V, 20%, X5R or X7S or similar, 0805, MLCC -> 22uF, Min. 25V, 20%, X5R or X7S or similar, 0805, MLCC
- C45: value 0.1uF_0603_16V -> 100nF_0402_16V; footprint 4ms_Capacitor:C_0603 -> 4ms_Capacitor:C_0402; symbol 4ms_Capacitor:0.1uF_0603_16V -> 4ms_Capacitor:100nF_0402_16V; JLCPCB ID C14663 -> C1525; Manufacturer AVX Corporation -> Murata; Manufacturer 2 (none) -> Yageo; Part Number 0603YC104KAT2A -> GCM155R71C104KA55D; Part Number 2 (none) -> CC0402KRX7R7BB104
- C6, C7: value 100nF_0402_16V -> 100nF_0603_16V; footprint 4ms_Capacitor:C_0402 -> 4ms_Capacitor:C_0603; symbol 4ms_Capacitor:100nF_0402_16V -> 4ms_Capacitor:100nF_0603_16V; JLCPCB ID C1525 -> C14663; Manufacturer Murata -> AVX Corporation; Part Number GCM155R71C104KA55D -> 0603YC104KAT2A
- C81, C98: value 10nF_0402_16V -> 10nF_0603_25V; footprint 4ms_Capacitor:C_0402 -> 4ms_Capacitor:C_0603; symbol 4ms_Capacitor:10nF_0402_16V -> 4ms_Capacitor:10nF_0603_25V; JLCPCB ID C15195 -> C57112; Manufacturer Yageo -> AVX Corporation; Part Number CC0402KRX7R7BB103 -> 06035C103KAT2A; Specifications 10nF, Min. 16V 10%, X7R or X5R or similar -> 10nF, Min 25V, 10%, X7R or similar
- POT1: value 16mm_CtrDet_10k -> 9mm_NoDet_100k_Knurled_Lined; footprint 4ms_Potentiometer:Pot_16mm_CtrDet_RV16AF-4A -> 4ms_Potentiometer:Pot_9mm_Knurl_NoDet; symbol 4ms_Potentiometer:16mm_CtrDet_10k -> 4ms_Potentiometer:9mm_NoDet_100k_Knurled_Lined; Display 10k -> 100k; Manufacturer Alpha Taiwan -> Song Huei; Part Number RV16AF-4A-15FW-B10k-3C -> R0904N-B100K L-25KQ/LWS; Specifications 10k Linear, 16mm pot, Center Detent, D-shaft -> 100k Linear, 9mm pot, No Detent, Knurled, Lined
- R1, R2: value 68R_0603 -> 68Ω_0603; symbol 4ms_Resistor:68R_0603 -> 4ms_Resistor_0603:68Ω_0603; Display 68R -> 68Ω; JLCPCB ID C27592 -> C126362; Production Stage (none) -> A; Specifications 68R, 1%, 1/10W, 0603 -> 68Ω, 1%, 1/10W, 0603
- R13, R5: value 47k_0402 -> 47k_0603; footprint 4ms_Resistor:R_0402 -> 4ms_Resistor:R_0603; symbol 4ms_Resistor_0402:47k_0402 -> 4ms_Resistor_0603:47k_0603; JLCPCB ID C93943 -> C105579; Part Number RC0402FR-0747KL -> RC0603FR-0747KL; Specifications 47k, 1%, 1/16W, 0402 -> 47k, 1%, 1/10W, 0603
- U11, U12, U8: value NJM2068 -> TL072H; symbol 4ms_IC:NJM2068 -> 4ms_IC:TL072H; JLCPCB ID (none) -> C4370341; Manufacturer NJR -> Texas Instruments; Part Number NJM2068V-TE1 -> TL072HIPWR; Specifications NJM2068 Dual Opamp -> Dual Opamp TSSOP-8
- U9: JLCPCB ID (none) -> C2651841
- V1: JLCPCB ID (none) -> C50754; JLCPCB ID 2 (none) -> C512090; JLCPCB ID 3 (none) -> C625398
Connections:
- net ADC-2: now also R2.2; no longer R1.2
- net ADC-3: now also R1.2; no longer R2.2
- net AUDIO_IN1: now also J10.1 (SIG)
- net AUDIO_IN2: now also J11.1 (SIG)
- net AUDIO_OUT1: now also J13.1 (SIG)
- net AUDIO_OUT2: now also J12.1 (SIG)
- net D10: no longer R47.1, U9.1 (MC/SCL/FMT)
- net D17: no longer R48.1, U9.2 (MD/SDA/DEMP)
- net D21: now also R48.1, U9.2 (MD/SDA/DEMP)
- net D3: no longer C81.1, D7.3 (AK), R13.2
- net D30: now also C81.1, D7.3 (AK), R13.2
- net D5: now also R47.1, U9.1 (MC/SCL/FMT)
- net GND: now also J10.2 (SHEILD), J10.3 (SW), J11.2 (SHEILD), J11.3 (SW), J12.2 (SHEILD), J13.2 (SHEILD), POT1.4 (Tab1), POT1.5 (Tab2); no longer C98.2
- net GNDADC: now also C98.2
- net -12VA renamed -12V
- no-connect marks 8 -> 10
Other:
- note added: "Example Audio Codec + Stereo In/Out"
- note added: "Example carrier board for mp153-devboard v0.1"
- note removed: "AUDIO"
- note removed: "DEVBOARD"
- note removed: "mp153"
- moved on the sheet: C147, C148, C149, C150, C152, C153, C3, C4, C41, C42, C44, C45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
