File: carrier board/p2/mp153-carrier-board.kicad_pcb (KiCad board)
At the start: 2 copper layers, 87.2 x 87.4 mm, 86 parts, among them J1 USB-C_Receptacle_Molex_217179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, J10 3.5mm_Mono_Switched_sm, J11 3.5mm_Mono_Switched_sm, J12 3.5mm_Mono_Switched_sm, J13 3.5mm_Mono_Switched_sm, J4 Socket_02x40_P0.4mm_W3.0mm_SMT, J5 3.5mm_Mono_Switched_sm, J6 Socket_02x40_P0.4mm_W3.0mm_SMT, J7 Eurorack_Power_16pin_Unshroud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, J9 3.5mm_Mono_Switched_sm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

Commit message: p2 carrier board: fixed position of headers
Parts:
- added Devboard-stand-in: mp153-dev-board-p1, 4ms_Symbol:4msLogo_3.8x1.7mm, B.Cu at (184.0, 120.8)
- added G***: LOGO, 4ms_Symbol:4msLogo_3.8x1.7mm, B.Cu at (183.7, 116.1)
- added H1: Spacer Nylon, fits 3mm hole, 4ms_Hardware:MountingHole_Generic_3mm, B.Cu at (237.7, 78.7)
- added H2: Spacer Nylon, fits 3mm hole, 4ms_Hardware:MountingHole_Generic_3mm, B.Cu at (223.5, 112.7)
- added H3: Spacer Nylon, fits 3mm hole, 4ms_Hardware:MountingHole_Generic_3mm, B.Cu at (187.7, 112.7)
- added H4: Spacer Nylon, fits 3mm hole, 4ms_Hardware:MountingHole_Generic_3mm, B.Cu at (187.7, 78.7)
- J4, J6: footprint mp153-devboard:Connector-80socket-P0.4mm-W3.0mm -> 4ms_Connector:Connector-80socket-P0.4mm-W3.0mm
- moved J1 23.5 mm to (248.4, 81.5)
- moved R3 23.5 mm to (242.2, 79.1)
- moved R4 22.4 mm to (242.2, 84.8)
- moved C81 12.4 mm to (180.9, 146.0)
- moved R13 11.9 mm to (179.1, 145.9)
- moved D7 10.3 mm to (176.2, 145.3)
- moved D1 4.95 mm to (172.6, 145.3)
- moved R5 4.93 mm to (169.8, 145.4)
- moved C1 4.72 mm to (168.5, 100.2)
- moved C2 4.72 mm to (174.6, 100.1)
- moved C8 4.72 mm to (170.3, 94.8)
- moved C98 4.72 mm to (169.0, 106.5)
- moved J4 4.72 mm to (187.1, 96.1)
- moved J6 4.72 mm to (237.1, 94.1)
- moved POT1 4.72 mm to (171.4, 85.9)
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Connections:
- C81 pad 1: /D30 -> /D28
- D7 pad 3: /D30 -> /D28
- R13 pad 2: /D30 -> /D28
- R2 pad 2: /ADC-2 -> /ADC-16
Routing:
- net /D30: track 60.4 -> 2.39 mm, vias 2 -> 0
- net /D28: track 2.39 -> 54.9 mm, vias 0 -> 2
- net +3V3: track 140.7 -> 173.2 mm
- net /D5: track 26.1 -> 46.4 mm, vias 0 -> 2
- net GND: track 575.4 -> 595.5 mm, vias 16 -> 22
- net /SAI_SD_B: track 23.1 -> 41.9 mm
- net /D21: track 27.4 -> 43.6 mm, vias 2 -> 0
- net /ADC-2: track 17.6 -> 2.39 mm, vias 2 -> 0
- net /ADC-16: track 2.39 -> 17.2 mm
- net /SAI_SD_A: track 30.8 -> 44.3 mm
- net /SAI_SCK: track 35.3 -> 47.3 mm, vias 0 -> 2
- net +12V: track 117.5 -> 129.1 mm
- net /SAI_FS: track 36.5 -> 47.2 mm, vias 2 -> 0
- net VREF+: track 16.6 -> 26.9 mm
- net /SAI_MCLK: track 34.1 -> 43.5 mm
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- added copper zone on B.Cu, net GND
Other:
- board text added: "1"
- board text added: "2"
- board text added: "79"
- board text added: "80"
- board text removed: "10k_0402"
- board text removed: "R28"
- board text removed: "R29"
- board text removed: "Reset"
