File: carrier board/p2/mp153-carrier-board.kicad_sch (KiCad schematic)
At the start: 86 parts, among them J1 USB-C_Receptacle_Molex_217179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, J10 3.5mm_Mono_Switched_sm, J11 3.5mm_Mono_Switched_sm, J12 3.5mm_Mono_Switched_sm, J13 3.5mm_Mono_Switched_sm, J4 Socket_02x40_P0.4mm_W3.0mm_SMT, J5 3.5mm_Mono_Switched_sm, J6 Socket_02x40_P0.4mm_W3.0mm_SMT, J7 Eurorack_Power_16pin_Unshroud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, J9 3.5mm_Mono_Switched_sm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

Commit message: p2 carrier board: fixed position of headers
Parts:
- J4, J6: footprint mp153-devboard:Connector-80socket-P0.4mm-W3.0mm -> 4ms_Connector:Connector-80socket-P0.4mm-W3.0mm
Connections:
- net ADC-16: now also R2.2
- net ADC-2: no longer R2.2
- net D28: now also C81.1, D7.3 (AK), R13.2
- net D30: no longer C81.1, D7.3 (AK), R13.2
Changed lines of the file:
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@@
 		)
 	)
-	(label "ADC-2"
+	(label "ADC-16"
 		(at 515.62 124.46 0)
 		(effects
@@
 		)
 	)
-	(label "D30"
+	(label "D28"
 		(at 476.25 226.06 0)
 		(effects
@@
 	)
 	(symbol
+		(lib_name "Socket_02x40_P0.4mm_W3.0mm_SMT_1")
 		(lib_id "4ms_Connector:Socket_02x40_P0.4mm_W3.0mm_SMT")
 		(at 198.12 115.57 0)
@@
 			)
 		)
-		(property "Footprint" "mp153-devboard:Connector-80socket-P0.4mm-W3.0mm"
+		(property "Footprint" "4ms_Connector:Connector-80socket-P0.4mm-W3.0mm"
 			(at 198.12 115.57 0)
 			(effects
@@
 			)
 		)
-		(property "Footprint" "mp153-devboard:Connector-80socket-P0.4mm-W3.0mm"
+		(property "Footprint" "4ms_Connector:Connector-80socket-P0.4mm-W3.0mm"
 			(at 43.18 115.57 0)
 			(effects
