File: carrier board/v0.2/mp153-carrier-board.kicad_sch (KiCad schematic)
At the start: 86 parts, among them J1 USB-C_Receptacle_Molex_217179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, J10 3.5mm_Mono_Switched_sm, J11 3.5mm_Mono_Switched_sm, J12 3.5mm_Mono_Switched_sm, J13 3.5mm_Mono_Switched_sm, J4 Socket_02x40_P0.4mm_W3.0mm_SMT, J5 3.5mm_Mono_Switched_sm, J6 Socket_02x40_P0.4mm_W3.0mm_SMT, J7 Eurorack_Power_16pin_Unshroud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, J9 3.5mm_Mono_Switched_sm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

Commit message: Move carrier board to v0.1 dir. Rename p2=>v0.2
Parts:
- removed R3, R4: 5.1k_0603, 4ms_Resistor:R_0603, symbol 4ms_Resistor_0603:5.1k_0603
- added C10, C9: 10uF_0805_16V_lowESR, 4ms_Capacitor:C_0805, symbol 4ms_Capacitor:10uF_0805_16V_lowESR
- added C70: 4.7uF_0402_6.3V, 4ms_Capacitor:C_0402, symbol 4ms_Capacitor:4.7uF_0402_6.3V
- added C79: 22uF_0603_6.3V, 4ms_Capacitor:C_0603, symbol 4ms_Capacitor:22uF_0603_6.3V
- added L1: FerriteBead_0603_0.8A_300mΩ, 4ms_Resistor:R_0603, symbol 4ms_Inductor:FerriteBead_0603_0.8A_300mΩ
- added U14: AP2411SN, 4ms_Package_QFP:DFN-6-1EP_2x2mm_P0.65mm_EP1x1.6mm, symbol 4ms_IC:AP2411SN
- added U3: FUSB302BMPX, Package_DFN_QFN:WQFN-14-1EP_2.5x2.5mm_P0.5mm_EP1.45x1.45mm, symbol 4ms_IC:FUSB302BMPX
Connections:
- net +5V: now also C79.2, U14.1 (IN), U3.3 (VDD), U3.4 (VDD)
- net D10: now also R47.1, U9.1 (MC/SCL/FMT)
- net D11: now also U3.5 (INT_N)
- net D17: now also R48.1, U9.2 (MD/SDA/DEMP)
- net D21: now also U3.7 (SDA); no longer R48.1, U9.2 (MD/SDA/DEMP)
- net D24: now also U14.3 (EN)
- net D5: now also U3.6 (SCL); no longer R47.1, U9.1 (MC/SCL/FMT)
- net GND: now also C10.2, C70.1, C79.1, C9.2, U14.2 (GND), U14.7 (EP), U3.15 (GND), U3.8 (GND), U3.9 (GND)
- net USB_VBUS_JACK: now also C9.1, L1.1, U3.2 (VBUS)
- net CC1: now reaches J1.A5 (CC1)
- net CC1: now also U3.10 (CC1), U3.11 (CC1)
- net CC2: now reaches J1.B5 (CC2)
- net CC2: now also U3.1 (CC2), U3.14 (CC2)
- new net USBSW_5V: C10.1, C70.2, L1.2, U14.5 (OUT)
- no-connect marks 10 -> 13
Other:
- note added: "Example carrier board for mp153-devboard v0.2"
- note added: "FUSB_INT"
- note added: "USB VBus +5V (switched on/off on demand) Max 500mA per USB specification"
- note added: "USB_5V_EN"
- note removed: "Example carrier board for mp153-devboard v0.1"
- moved on the sheet: C1, C2, C3, C4, C49, C5, C51, C6, C7, C8, C81, C98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

Commit message: carrier board: fix-it notes for v0.2
Other:
- note added: "Fixes for v0.2 (to be in v0.3): - Don't use I2C3 since it conflicts with SD Card - Swap USB + and -"
Changed lines of the file:
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@@
+		)
+	)
+	(text "Fixes for v0.2 (to be in v0.3):\n- Don't use I2C3 since it conflicts with SD Card\n- Swap USB + and -"
+		(exclude_from_sim no)
+		(at 148.844 -14.478 0)
+		(effects
+			(font
+				(size 1.905 1.905)
+			)
+			(justify left)
 		)
 	)
