File: v0.2/mp153-devboard.kicad_sch (KiCad schematic)
At the start: 122 parts, among them CON1 microSDCon_SMT_104031-0811, J1 Pins_02x40_P0.4mm_W3.0mm_SMT, J2 Pins_02x40_P0.4mm_W3.0mm_SMT, J3 USB-C_Receptacle_Molex_217179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, J4 Pins_02x04_RightAngle_P2.54mm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, J5 Conn_01x02, J6 Pins_02x05_P1.27mm_SMT, U13 NCP51460SN33, U14 DDR3L-RAM-4Gb_MT41K256M16TW, U15 AP6230xZ6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

Commit message: v0.2: Update AP62301Z6 part numbers
Parts:
- U15, U16, U17: Part Number AP62301Z6 -> AP62301Z6-7; Part Number 2 AP62300Z6 -> AP62300Z6-7; Part Number 3 AP62300TZ6 -> AP62300TZ6-7
Changed lines of the file:
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@@
 			)
 		)
-		(property "Description" ""
+		(property "Description" "3A, 750kHz Buck DC/DC Converter, VinMax>=12V, SOT-563"
 			(at 408.94 219.71 0)
 			(effects
@@
 			)
 		)
-		(property "Part Number" "AP62301Z6"
+		(property "Part Number" "AP62301Z6-7"
 			(at 408.94 241.3 0)
 			(effects
@@
 			)
 		)
-		(property "Part Number 2" "AP62300Z6"
+		(property "Part Number 2" "AP62300Z6-7"
 			(at 408.94 238.76 0)
 			(effects
@@
 			)
 		)
-		(property "Part Number 3" "AP62300TZ6"
+		(property "Part Number 3" "AP62300TZ6-7"
 			(at 408.94 236.22 0)
 			(effects
@@
 			)
 		)
-		(property "Description" ""
+		(property "Description" "3A, 750kHz Buck DC/DC Converter, VinMax>=12V, SOT-563"
 			(at 408.94 176.53 0)
 			(effects
@@
 			)
 		)
-		(property "Part Number" "AP62301Z6"
+		(property "Part Number" "AP62301Z6-7"
 			(at 408.94 198.12 0)
 			(effects
@@
 			)
 		)
-		(property "Part Number 2" "AP62300Z6"
+		(property "Part Number 2" "AP62300Z6-7"
 			(at 408.94 195.58 0)
 			(effects
@@
 			)
 		)
-		(property "Part Number 3" "AP62300TZ6"
+		(property "Part Number 3" "AP62300TZ6-7"
 			(at 408.94 193.04 0)
 			(effects
@@
 			)
 		)
-		(property "Description" ""
+		(property "Description" "3A, 750kHz Buck DC/DC Converter, VinMax>=12V, SOT-563"
 			(at 408.94 134.62 0)
 			(effects
@@
 			)
 		)
-		(property "Part Number" "AP62301Z6"
+		(property "Part Number" "AP62301Z6-7"
 			(at 408.94 156.21 0)
 			(effects
@@
 			)
 		)
-		(property "Part Number 2" "AP62300Z6"
+		(property "Part Number 2" "AP62300Z6-7"
 			(at 408.94 153.67 0)
 			(effects
@@
 			)
 		)
-		(property "Part Number 3" "AP62300TZ6"
+		(property "Part Number 3" "AP62300TZ6-7"
 			(at 408.94 151.13 0)
 			(effects

Commit message: TODO note for v0.2 board
Other:
- note added: "TODO for v0.3: Connect PE14 or PG7 to pins (LCD_CLK)"
Changed lines of the file:
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@@
+		)
+	)
+	(text "TODO for v0.3:\nConnect PE14 or PG7 to pins (LCD_CLK)"
+		(exclude_from_sim no)
+		(at 153.67 32.258 0)
+		(effects
+			(font
+				(size 2.54 2.54)
+			)
+			(justify left bottom)
 		)
 	)
