File: carrier board/v0.4/mp153-carrier-board.kicad_sch (KiCad schematic)
At the start: 99 parts, among them J1 USB-C_Receptacle_Molex_217179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, J10 3.5mm_Mono_Switched_sm, J11 3.5mm_Mono_Switched_sm, J12 3.5mm_Mono_Switched_sm, J13 3.5mm_Mono_Switched_sm, J2 Eurorack_Power_10pin_Shrouded, J5 3.5mm_Mono_Switched_sm, J9 3.5mm_Mono_Switched_sm, U1 TL072H, U11 TL072H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

Commit message: carrier-board v0.4: notes and updates
Parts:
- J3: footprint mp153-devboard:mp153-devboard-v0.1-sockets_B -> 4ms_Connector_Card:mp153-devboard-sockets_B; symbol mp153-devboard:mp153-devboard-v0.1-guide-B -> 4ms_IC:mp153-devboard-v0.2-socket-B; Alt JLCPCB ID (none) -> C312960; Alt Part Number (none) -> DF40C-80DS-0.4V(51); JLCPCB ID (none) -> C2858577; Manufacturer (none) -> Hirose; Part Number (none) -> DF40HC(3.0)-80DS-0.4V(51)
- J4: footprint mp153-devboard:mp153-devboard-v0.1-sockets_A -> 4ms_Connector_Card:mp153-devboard-sockets_A; symbol mp153-devboard:mp153-devboard-v0.1-guide-A -> 4ms_IC:mp153-devboard-v0.2-socket-A; Alt JLCPCB ID (none) -> C312960; Alt Part Number (none) -> DF40C-80DS-0.4V(51); JLCPCB ID (none) -> C2858577; Manufacturer (none) -> Hirose; Part Number (none) -> DF40HC(3.0)-80DS-0.4V(51)
Connections:
- no-connect marks 49 -> 50
Changed lines of the file:
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@@
 	)
 	(no_connect
+		(at 66.04 99.06)
+	)
+	(no_connect
 		(at 205.74 251.46)
 	)
@@
 	)
 	(symbol
-		(lib_id "mp153-devboard:mp153-devboard-v0.1-guide-B")
+		(lib_id "4ms_IC:mp153-devboard-v0.2-socket-B")
 		(at 128.27 100.33 0)
 		(unit 1)
@@
 			)
 		)
-		(property "Footprint" "mp153-devboard:mp153-devboard-v0.1-sockets_B"
+		(property "Footprint" "4ms_Connector_Card:mp153-devboard-sockets_B"
 			(at 128.27 157.48 0)
 			(effects
@@
 			)
 		)
-		(property "Description" "Socket B for an mp153-devboard v0.1 (requires Socket A)"
+		(property "Description" "Socket B for an mp153-devboard v0.2 (requires Socket A)"
 			(at 128.27 162.56 0)
 			(effects
@@
 			)
 		)
+		(property "Manufacturer" "Hirose"
+			(at 128.27 100.33 0)
+			(effects
+				(font
+					(size 1.27 1.27)
+				)
+				(hide yes)
+			)
+		)
+		(property "Part Number" "DF40HC(3.0)-80DS-0.4V(51) "
+			(at 128.27 100.33 0)
+			(effects
+				(font
+					(size 1.27 1.27)
+				)
+				(hide yes)
+			)
+		)
+		(property "Alt Part Number" "DF40C-80DS-0.4V(51)"
+			(at 128.27 100.33 0)
+			(effects
+				(font
+					(size 1.27 1.27)
+				)
+				(hide yes)
+			)
+		)
+		(property "JLCPCB ID" "C2858577"
+			(at 128.27 100.33 0)
+			(effects
+				(font
+					(size 1.27 1.27)
+				)
+				(hide yes)
+			)
+		)
+		(property "Alt JLCPCB ID" "C312960"
+			(at 128.27 100.33 0)
+			(effects
+				(font
+					(size 1.27 1.27)
+				)
+				(hide yes)
+			)
+		)
 		(pin "B64"
 		)
@@
 	)
 	(symbol
-		(lib_id "mp153-devboard:mp153-devboard-v0.1-guide-A")
+		(lib_id "4ms_IC:mp153-devboard-v0.2-socket-A")
 		(at 90.17 100.33 0)
 		(unit 1)
@@
 			)
 		)
-		(property "Footprint" "mp153-devboard:mp153-devboard-v0.1-sockets_A"
+		(property "Footprint" "4ms_Connector_Card:mp153-devboard-sockets_A"
 			(at 90.17 157.48 0)
 			(effects
@@
 			)
 		)
-		(property "Description" "Socket A for an mp153-devboard v0.1 (requires Socket B)"
+		(property "Description" "Socket A for an mp153-devboard v0.2 (requires Socket B)"
 			(at 90.17 162.56 0)
 			(effects
 				(font
+					(size 1.27 1.27)
+				)
+				(hide yes)
+			)
+		)
+		(property "Manufacturer" "Hirose"
+			(at 90.17 100.33 0)
+			(effects
+				(font
+					(size 1.27 1.27)
+				)
+				(hide yes)
+			)
+		)
+		(property "Part Number" "DF40HC(3.0)-80DS-0.4V(51) "
+			(at 90.17 100.33 0)
+			(effects
+				(font
+					(size 1.27 1.27)
+				)
+				(hide yes)
+			)
+		)
+		(property "Alt Part Number" "DF40C-80DS-0.4V(51)"
+			(at 90.17 100.33 0)
+			(effects
+				(font
+					(size 1.27 1.27)
+				)
+				(hide yes)
+			)
+		)
+		(property "JLCPCB ID" "C2858577"
+			(at 90.17 100.33 0)
+			(effects
+				(font
+					(size 1.27 1.27)
+				)
+				(hide yes)
+			)
+		)
+		(property "Alt JLCPCB ID" "C312960"
+			(at 90.17 100.33 0)
+			(effects
+				(font
