File: carrier-breakout/v0.1/mp153-carrier-board.kicad_pcb (KiCad board)
At the start: 2 copper layers, 110 x 125 mm, 102 parts, among them J1 USB-C_Receptacle_Molex_217179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, J10 3.5mm_Mono_Switched_sm, J11 3.5mm_Mono_Switched_sm, J12 3.5mm_Mono_Switched_sm, J13 3.5mm_Mono_Switched_sm, J2 Eurorack_Power_10pin_Shrouded, J6 Pins_02x40_P2.54mm_TH, J7 Pins_02x40_P2.54mm_TH, U11 TL072H, U12 TL072H, U13 AP6230xZ6, U14 AP2411SN, U3 FUSB302BMPX, U8 TL072H, U9 PCM3060PW

Commit message: Removed redundant ADC net labels
Connections:
- net /ADC_10 renamed /B52
- net /ADC_11 renamed /B38
- net /ADC_12 renamed /B36
- net /ADC_13 renamed /B34
- net /ADC_14 renamed /B44
- net /ADC_15 renamed /B32
- net /ADC_16 renamed /B30
- net /ADC_17 renamed /B40
- net /ADC_18 renamed /B60
- net /ADC_19 renamed /B56
- net /ADC_2 renamed /B62
- net /ADC_3 renamed /B58
- net /ADC_4 renamed /B50
- net /ADC_5 renamed /B46
- net /ADC_7 renamed /B54
- net /ADC_8 renamed /B48
- net /ADC_9 renamed /B42
Changed lines of the file:
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@@
 	(net 71 "Net-(U13-SW)")
 	(net 72 "Net-(U13-FB)")
-	(net 73 "/ADC_9")
+	(net 73 "/B42")
 	(net 74 "/B2")
 	(net 75 "/B4")
 	(net 76 "/B16")
-	(net 77 "/ADC_16")
-	(net 78 "/ADC_5")
-	(net 79 "/ADC_3")
-	(net 80 "/ADC_13")
-	(net 81 "/ADC_12")
-	(net 82 "/ADC_10")
+	(net 77 "/B30")
+	(net 78 "/B46")
+	(net 79 "/B58")
+	(net 80 "/B34")
+	(net 81 "/B36")
+	(net 82 "/B52")
 	(net 83 "/B12")
 	(net 84 "/B76")
-	(net 85 "/ADC_7")
-	(net 86 "/ADC_4")
+	(net 85 "/B54")
+	(net 86 "/B50")
 	(net 87 "/B10")
 	(net 88 "/B22")
-	(net 89 "/ADC_15")
+	(net 89 "/B32")
 	(net 90 "/B6")
-	(net 91 "/ADC_8")
-	(net 92 "/ADC_14")
+	(net 91 "/B48")
+	(net 92 "/B44")
 	(net 93 "/B74")
 	(net 94 "/B20")
-	(net 95 "/ADC_18")
-	(net 96 "/ADC_11")
+	(net 95 "/B60")
+	(net 96 "/B38")
 	(net 97 "/B72")
 	(net 98 "/B14")
-	(net 99 "/ADC_19")
+	(net 99 "/B56")
 	(net 100 "/B8")
-	(net 101 "/ADC_2")
+	(net 101 "/B62")
 	(net 102 "/B18")
 	(net 103 "/B70")
-	(net 104 "/ADC_17")
+	(net 104 "/B40")
 	(net 105 "/A19")
 	(net 106 "/A61")
@@
 			(layers "*.Cu" "*.Mask")
 			(remove_unused_layers no)
-			(net 77 "/ADC_16")
+			(net 77 "/B30")
 			(pinfunction "Pin_29")
 			(pintype "passive")
@@
 			(layers "*.Cu" "*.Mask")
 			(remove_unused_layers no)
-			(net 77 "/ADC_16")
+			(net 77 "/B30")
 			(pinfunction "Pin_30")
 			(pintype "passive")
@@
 			(layers "*.Cu" "*.Mask")
 			(remove_unused_layers no)
-			(net 89 "/ADC_15")
+			(net 89 "/B32")
 			(pinfunction "Pin_31")
 			(pintype "passive")
@@
 			(layers "*.Cu" "*.Mask")
 			(remove_unused_layers no)
-			(net 89 "/ADC_15")
+			(net 89 "/B32")
 			(pinfunction "Pin_32")
 			(pintype "passive")
@@
 			(layers "*.Cu" "*.Mask")
 			(remove_unused_layers no)
-			(net 80 "/ADC_13")
+			(net 80 "/B34")
 			(pinfunction "Pin_33")
 			(pintype "passive")
@@
 			(layers "*.Cu" "*.Mask")
 			(remove_unused_layers no)
-			(net 80 "/ADC_13")
+			(net 80 "/B34")
 			(pinfunction "Pin_34")
 			(pintype "passive")
@@
 			(layers "*.Cu" "*.Mask")
 			(remove_unused_layers no)
-			(net 81 "/ADC_12")
+			(net 81 "/B36")
 			(pinfunction "Pin_35")
 			(pintype "passive")
@@
 			(layers "*.Cu" "*.Mask")
 			(remove_unused_layers no)
-			(net 81 "/ADC_12")
+			(net 81 "/B36")
 			(pinfunction "Pin_36")
 			(pintype "passive")
@@
 			(layers "*.Cu" "*.Mask")
 			(remove_unused_layers no)
-			(net 96 "/ADC_11")
+			(net 96 "/B38")
 			(pinfunction "Pin_37")
 			(pintype "passive")
@@
 			(layers "*.Cu" "*.Mask")
 			(remove_unused_layers no)
-			(net 96 "/ADC_11")
+			(net 96 "/B38")
 			(pinfunction "Pin_38")
 			(pintype "passive")
@@
 			(layers "*.Cu" "*.Mask")
 			(remove_unused_layers no)
-			(net 104 "/ADC_17")
+			(net 104 "/B40")
 			(pinfunction "Pin_39")
 			(pintype "passive")
@@
 			(layers "*.Cu" "*.Mask")
 			(remove_unused_layers no)
-			(net 104 "/ADC_17")
+			(net 104 "/B40")
 			(pinfunction "Pin_40")
 			(pintype "passive")
@@
 			(layers "*.Cu" "*.Mask")
 			(remove_unused_layers no)
-			(net 73 "/ADC_9")
+			(net 73 "/B42")
 			(pinfunction "Pin_41")
 			(pintype "passive")
@@
 			(layers "*.Cu" "*.Mask")
 			(remove_unused_layers no)
-			(net 73 "/ADC_9")
+			(net 73 "/B42")
 			(pinfunction "Pin_42")
 			(pintype "passive")
@@
 			(layers "*.Cu" "*.Mask")
 			(remove_unused_layers no)
-			(net 92 "/ADC_14")
+			(net 92 "/B44")
 			(pinfunction "Pin_43")
 			(pintype "passive")
@@
 			(layers "*.Cu" "*.Mask")
 			(remove_unused_layers no)
-			(net 92 "/ADC_14")
+			(net 92 "/B44")
 			(pinfunction "Pin_44")
 			(pintype "passive")
@@
 			(layers "*.Cu" "*.Mask")
 			(remove_unused_layers no)
-			(net 78 "/ADC_5")
+			(net 78 "/B46")
 			(pinfunction "Pin_45")
 			(pintype "passive")
@@
 			(layers "*.Cu" "*.Mask")
 			(remove_unused_layers no)
-			(net 78 "/ADC_5")
+			(net 78 "/B46")
 			(pinfunction "Pin_46")
 			(pintype "passive")
@@
 			(layers "*.Cu" "*.Mask")
 			(remove_unused_layers no)
-			(net 91 "/ADC_8")
+			(net 91 "/B48")
 			(pinfunction "Pin_47")
 			(pintype "passive")
@@
 			(layers "*.Cu" "*.Mask")
 			(remove_unused_layers no)
-			(net 91 "/ADC_8")
+			(net 91 "/B48")
 			(pinfunction "Pin_48")
 			(pintype "passive")
@@
 			(layers "*.Cu" "*.Mask")
 			(remove_unused_layers no)
-			(net 86 "/ADC_4")
+			(net 86 "/B50")
 			(pinfunction "Pin_49")
 			(pintype "passive")
@@
 			(layers "*.Cu" "*.Mask")
 			(remove_unused_layers no)
-			(net 86 "/ADC_4")
+			(net 86 "/B50")
 			(pinfunction "Pin_50")
 			(pintype "passive")
@@
 			(layers "*.Cu" "*.Mask")
 			(remove_unused_layers no)
-			(net 82 "/ADC_10")
+			(net 82 "/B52")
 			(pinfunction "Pin_51")
 			(pintype "passive")
@@
 			(layers "*.Cu" "*.Mask")
 			(remove_unused_layers no)
-			(net 82 "/ADC_10")
+			(net 82 "/B52")
 			(pinfunction "Pin_52")
 			(pintype "passive")
@@
 			(layers "*.Cu" "*.Mask")
 			(remove_unused_layers no)
-			(net 85 "/ADC_7")
+			(net 85 "/B54")
 			(pinfunction "Pin_53")
 			(pintype "passive")
@@
 			(layers "*.Cu" "*.Mask")
 			(remove_unused_layers no)
-			(net 85 "/ADC_7")
+			(net 85 "/B54")
 			(pinfunction "Pin_54")
 			(pintype "passive")
@@
 			(layers "*.Cu" "*.Mask")
 			(remove_unused_layers no)
-			(net 99 "/ADC_19")
+			(net 99 "/B56")
 			(pinfunction "Pin_55")
 			(pintype "passive")
@@
 			(layers "*.Cu" "*.Mask")
 			(remove_unused_layers no)
-			(net 99 "/ADC_19")
+			(net 99 "/B56")
 			(pinfunction "Pin_56")
 			(pintype "passive")
@@
 			(layers "*.Cu" "*.Mask")
 			(remove_unused_layers no)
-			(net 79 "/ADC_3")
+			(net 79 "/B58")
 			(pinfunction "Pin_57")
 			(pintype "passive")
@@
 			(layers "*.Cu" "*.Mask")
 			(remove_unused_layers no)
-			(net 79 "/ADC_3")
+			(net 79 "/B58")
 			(pinfunction "Pin_58")
 			(pintype "passive")
@@
 			(layers "*.Cu" "*.Mask")
 			(remove_unused_layers no)
-			(net 95 "/ADC_18")
+			(net 95 "/B60")
 			(pinfunction "Pin_59")
 			(pintype "passive")
@@
 			(layers "*.Cu" "*.Mask")
 			(remove_unused_layers no)
-			(net 95 "/ADC_18")
+			(net 95 "/B60")
 			(pinfunction "Pin_60")
 			(pintype "passive")
@@
 			(layers "*.Cu" "*.Mask")
 			(remove_unused_layers no)
-			(net 101 "/ADC_2")
+			(net 101 "/B62")
 			(pinfunction "Pin_61")
 			(pintype "passive")
@@
 			(layers "*.Cu" "*.Mask")
 			(remove_unused_layers no)
-			(net 101 "/ADC_2")
+			(net 101 "/B62")
 			(pinfunction "Pin_62")
 			(pintype "passive")
@@
 			(size 0.2 3.78)
 			(layers "F.Cu" "F.Mask" "F.Paste")
-			(net 77 "/ADC_16")
+			(net 77 "/B30")
 			(pinfunction "PA0")
 			(pintype "passive")
@@
 			(size 0.2 3.78)
 			(layers "F.Cu" "F.Mask" "F.Paste")
-			(net 89 "/ADC_15")
+			(net 89 "/B32")
 			(pinfunction "PA3")
 			(pintype "passive")
@@
 			(size 0.2 3.78)
 			(layers "F.Cu" "F.Mask" "F.Paste")
-			(net 80 "/ADC_13")
+			(net 80 "/B34")
 			(pinfunction "PC3")
 			(pintype "passive")
@@
 			(size 0.2 3.78)
 			(layers "F.Cu" "F.Mask" "F.Paste")
-			(net 81 "/ADC_12")
+			(net 81 "/B36")
 			(pinfunction "PC2")
 			(pintype "passive")
@@
 			(size 0.2 3.78)
 			(layers "F.Cu" "F.Mask" "F.Paste")
-			(net 96 "/ADC_11")
+			(net 96 "/B38")
 			(pinfunction "PC1")
 			(pintype "passive")
@@
 			(size 0.2 3.78)
 			(layers "F.Cu" "F.Mask" "F.Paste")
-			(net 104 "/ADC_17")
+			(net 104 "/B40")
 			(pinfunction "PA1")
 			(pintype "passive")
@@
 			(size 0.2 3.78)
 			(layers "F.Cu" "F.Mask" "F.Paste")
-			(net 73 "/ADC_9")
+			(net 73 "/B42")
 			(pinfunction "PB0")
 			(pintype "passive")
@@
 			(size 0.2 3.78)
 			(layers "F.Cu" "F.Mask" "F.Paste")
-			(net 92 "/ADC_14")
+			(net 92 "/B44")
 			(pinfunction "PA2")
 			(pintype "passive")
@@
 			(size 0.2 3.78)
 			(layers "F.Cu" "F.Mask" "F.Paste")
-			(net 78 "/ADC_5")
+			(net 78 "/B46")
 			(pinfunction "PB1")
 			(pintype "passive")
@@
 			(size 0.2 3.78)
 			(layers "F.Cu" "F.Mask" "F.Paste")
-			(net 91 "/ADC_8")
+			(net 91 "/B48")
 			(pinfunction "PC5")
 			(pintype "passive")
@@
 			(size 0.2 3.78)
 			(layers "F.Cu" "F.Mask" "F.Paste")
-			(net 86 "/ADC_4")
+			(net 86 "/B50")
 			(pinfunction "PC4")
 			(pintype "passive")
@@
 			(size 0.2 3.78)
 			(layers "F.Cu" "F.Mask" "F.Paste")
-			(net 82 "/ADC_10")
+			(net 82 "/B52")
 			(pinfunction "PC0")
 			(pintype "passive")
@@
 			(size 0.2 3.78)
 			(layers "F.Cu" "F.Mask" "F.Paste")
-			(net 85 "/ADC_7")
+			(net 85 "/B54")
 			(pinfunction "PA7")
 			(pintype "passive")
@@
 			(size 0.2 3.78)
 			(layers "F.Cu" "F.Mask" "F.Paste")
-			(net 99 "/ADC_19")
+			(net 99 "/B56")
 			(pinfunction "PA5")
 			(pintype "passive")
@@
 			(size 0.2 3.78)
 			(layers "F.Cu" "F.Mask" "F.Paste")
-			(net 79 "/ADC_3")
+			(net 79 "/B58")
 			(pinfunction "PA6")
 			(pintype "passive")
@@
 			(size 0.2 3.78)
 			(layers "F.Cu" "F.Mask" "F.Paste")
-			(net 95 "/ADC_18")
+			(net 95 "/B60")
 			(pinfunction "PA4")
 			(pintype "passive")
@@
 			(size 0.2 3.78)
 			(layers "F.Cu" "F.Mask" "F.Paste")
-			(net 101 "/ADC_2")
+			(net 101 "/B62")
 			(pinfunction "PF11")
 			(pintype "passive")

Commit message: carrier-breakout cleanup:
- Fix nets with two names
- Fix some silk overlap DRC warning for components too close
- Add more space for pins names to fix DRC warnings for silk sizes
- Remove empty boxes on silk
- Space out jumpers that we may have to cut with an exacto (more space = easier to cut)
- Added jumper for USB_5V_ENABLE, and pull-down to prevent floating when jumper is cut
Parts:
- removed C70: 4.7uF_0402_6.3V, 4ms_Capacitor:C_0402
- added JP16: SolderJumper_2_Open, 4ms_SolderJumper:JUMPER_SMD_1x2_tiny, F.Cu at (-15.8, -40.3)
- added R3: 10k_0402, 4ms_Resistor:R_0402, F.Cu at (-13.6, -38.5)
- C11, C3, C41, C45: value 100nF_0402_16V -> 100nF_0402_50V
- C74: value 22uF_1206_25V -> 22uF_0805_25V
- moved JP8 10.4 mm to (0.30, 2.97)
- moved JP10 9.32 mm to (6.04, 3.12)
- moved JP5 8.92 mm to (0.30, 5.97)
- moved JP9 8.20 mm to (6.04, 6.12)
- moved JP6 7.42 mm to (0.30, 8.97)
- moved JP4 5.92 mm to (0.30, 12.0)
- moved JP11 5.45 mm to (-23.8, -49.4)
- moved JP2 4.39 mm to (0.26, 15.0)
- moved JP15 3.94 mm to (-22.3, -47.5)
- moved C6 3.19 mm to (21.3, -40.6)
- moved JP12 3.13 mm to (-17.6, -41.4)
- moved C7 3.11 mm to (14.0, -40.7)
- moved C5 3.04 mm to (13.9, -44.4)
- moved C4 3.00 mm to (22.0, -44.5)
- moved JP14 2.94 mm to (-20.5, -44.8)
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Connections:
- net /A71 renamed /USB_VBUS_JACK
- net /A75 renamed /USB_HS_D+
- net /A77 renamed /USB_HS_D-
- U14 pad 3: /A57 -> /USB_5V_ENABLE
Routing:
- net /A51: track 78.6 -> 69.7 mm
- net /A61: track 122.0 -> 113.8 mm
- net /A45: track 74.9 -> 67.5 mm
- net +3V3: track 141.6 -> 134.4 mm
- net /USB_5V_ENABLE: track 0.00 -> 7.17 mm
- net /A57: track 77.3 -> 70.1 mm
- net /A59: track 120.3 -> 113.3 mm
- net /A47: track 78.2 -> 72.2 mm
- net /SAI_SD_B: track 21.4 -> 27.3 mm
- net /5V_FUSB: track 5.17 -> 10.7 mm
- net /A43: track 76.9 -> 72.2 mm
- net /FUSB_INT: track 5.34 -> 9.50 mm
- net +5V: track 172.5 -> 176.5 mm
- net /SAI_FS: track 28.1 -> 32.1 mm
- net /A49: track 84.3 -> 80.9 mm
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- removed copper zone on B.Cu, net GND
- removed copper zone on F.Cu, net GND
Other:
- board size 110 x 125 mm -> 123.7 x 125 mm
