File: v0.3-mp133/mp133-devboard.kicad_sch (KiCad schematic)
At the start: 146 parts, among them CON1 microSDCon_SMT_104031-0811, J1 Pins_02x40_P0.4mm_W3.0mm_SMT, J2 Pins_02x40_P0.4mm_W3.0mm_SMT, J3 USB-C_Receptacle_Molex_217179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, J4 Pins_02x04_RightAngle_P2.54mm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, J5 Conn_01x02, J6 Pins_02x05_P1.27mm_SMT, U13 NCP51460SN33, U14 DDR3L-RAM-4Gb_MT41K256M16TW, U15 AP6230xZ6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

Commit message: mp133: WIP routing and pin assignment
Connections:
- net DEBUG0: no longer U2.C14 (PB3)
- net PA10: now also J1.63 (Pin_63), J1.64 (Pin_64)
- net PB8: now also J1.3 (Pin_3), J1.4 (Pin_4)
- net PD7: no longer J2.10 (Pin_10), J2.9 (Pin_9)
- net UART_TX: no longer U2.A2 (PA9)
- net PH8: now reaches U2.E3 (PH8)
- net PH8: now also J2.10 (Pin_10), J2.9 (Pin_9)
- net PA9: now reaches J2.5 (Pin_5), J2.6 (Pin_6)
- net PA9: now also U2.A2 (PA9)
- net PB15: now reaches J1.5 (Pin_5), J1.6 (Pin_6)
- net PB15: now also U2.B15 (PB15)
Other:
- note added: "TIM1_CH3"
- note added: "UART_RX, I2C_SCL"
Changed lines of the file:
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@@
 	(text "SAI2_SCK"
 		(exclude_from_sim no)
-		(at 161.29 72.136 0)
+		(at 149.098 76.708 0)
 		(effects
 			(font
@@
 		)
 	)
-	(text "SAI2_SD_B"
-		(exclude_from_sim no)
-		(at 93.98 69.596 0)
-		(effects
-			(font
-				(size 1.27 1.27)
-			)
-			(justify right bottom)
-		)
-	)
 	(text "I2C3_SDA"
 		(exclude_from_sim no)
-		(at 132.842 419.1 0)
+		(at 294.64 411.48 0)
 		(effects
 			(font
 				(size 1.27 1.27)
 			)
-			(justify left bottom)
+			(justify right bottom)
 		)
 	)
@@
 	(text "SPI3_MOSI"
 		(exclude_from_sim no)
-		(at 3.556 70.866 0)
+		(at 3.556 70.358 0)
 		(effects
 			(font
@@
 		)
 	)
+	(text "SPI3_MOSI"
+		(exclude_from_sim no)
+		(at 49.53 439.42 0)
+		(effects
+			(font
+				(size 1.27 1.27)
+			)
+			(justify left bottom)
+		)
+	)
 	(text "SD_CARD_DETECT"
 		(exclude_from_sim no)
@@
 		)
 	)
+	(text "TIM1_CH3"
+		(exclude_from_sim no)
+		(at 48.768 383.54 0)
+		(effects
+			(font
+				(size 1.27 1.27)
+			)
+			(justify left bottom)
+		)
+	)
 	(text "ADC-5"
 		(exclude_from_sim no)
@@
 		)
 	)
+	(text "UART_RX, I2C_SCL"
+		(exclude_from_sim no)
+		(at 217.678 69.596 0)
+		(effects
+			(font
+				(size 1.27 1.27)
+			)
+			(justify left bottom)
+		)
+	)
 	(text "I2C1_SDA"
 		(exclude_from_sim no)
@@
 		)
 	)
+	(text "SPI3_MOSI"
+		(exclude_from_sim no)
+		(at 76.2 72.39 0)
+		(effects
+			(font
+				(size 1.27 1.27)
+			)
+			(justify right bottom)
+		)
+	)
 	(text "          BOOT0  BOOT2\nSD Card    On     On\nFlash      On    Off\nDebugger   Off    On"
 		(exclude_from_sim no)
@@
 		)
 	)
+	(text "TIM1_CH3"
+		(exclude_from_sim no)
+		(at 76.962 146.05 0)
+		(effects
+			(font
+				(size 1.27 1.27)
+			)
+			(justify right bottom)
+		)
+	)
 	(text "ADC-9"
 		(exclude_from_sim no)
@@
 		)
 	)
-	(text "TIM PWM"
-		(exclude_from_sim no)
-		(at 26.67 145.796 0)
-		(effects
-			(font
-				(size 1.27 1.27)
-			)
-			(justify left bottom)
-		)
-	)
 	(text "SAI1_SCK"
 		(exclude_from_sim no)
@@
 	(wire
 		(pts
+			(xy 271.78 411.48) (xy 299.72 411.48)
+		)
+		(stroke
+			(width 0)
+			(type default)
+		)
+	)
+	(wire
+		(pts
 			(xy 528.32 374.65) (xy 528.32 377.19)
 		)
@@
 	(wire
 		(pts
-			(xy 55.88 408.94) (xy 69.85 408.94)
-		)
-		(stroke
-			(width 0)
-			(type default)
-		)
-	)
-	(wire
-		(pts
 			(xy 204.47 609.6) (xy 184.15 609.6)
 		)
@@
 	(wire
 		(pts
-			(xy 55.88 381) (xy 69.85 381)
-		)
-		(stroke
-			(width 0)
-			(type default)
-		)
-	)
-	(wire
-		(pts
 			(xy 323.85 400.05) (xy 351.79 400.05)
 		)
@@
 	(wire
 		(pts
+			(xy 43.18 381) (xy 69.85 381)
+		)
+		(stroke
+			(width 0)
+			(type default)
+		)
+	)
+	(wire
+		(pts
 			(xy 458.47 264.16) (xy 458.47 259.08)
 		)
@@
 	(wire
 		(pts
+			(xy 43.18 408.94) (xy 69.85 408.94)
+		)
+		(stroke
+			(width 0)
+			(type default)
+		)
+	)
+	(wire
+		(pts
 			(xy 54.61 544.83) (xy 39.37 544.83)
 		)
@@
 	(wire
 		(pts
+			(xy 43.18 439.42) (xy 69.85 439.42)
+		)
+		(stroke
+			(width 0)
+			(type default)
+		)
+	)
+	(wire
+		(pts
 			(xy 187.96 97.79) (xy 201.93 97.79)
 		)
@@
 		)
 	)
+	(label "PB8"
+		(at 82.55 69.85 180)
+		(effects
+			(font
+				(size 1.27 1.27)
+			)
+			(justify right bottom)
+		)
+	)
 	(label "DDR_A8"
 		(at 113.03 552.45 180)
@@
 		)
 	)
-	(label "UART_TX"
-		(at 55.88 381 0)
-		(effects
-			(font
-				(size 1.27 1.27)
-			)
-			(justify left bottom)
-		)
-	)
 	(label "DDR_BA2"
 		(at 184.15 629.92 0)
@@
 		)
 	)
+	(label "PH8"
+		(at 173.99 77.47 0)
+		(effects
+			(font
+				(size 1.27 1.27)
+			)
+			(justify left bottom)
+		)
+	)
 	(label "FLASH_CLK"
 		(at 153.67 278.13 180)
@@
 		)
 	)
+	(label "PH8"
+		(at 299.72 411.48 180)
+		(effects
+			(font
+				(size 1.27 1.27)
+			)
+			(justify right bottom)
+		)
+	)
 	(label "DDR_DQ11"
 		(at 39.37 562.61 0)
@@
 		)
 	)
+	(label "PA9"
+		(at 173.99 72.39 0)
+		(effects
+			(font
+				(size 1.27 1.27)
+			)
+			(justify left bottom)
+		)
+	)
 	(label "DDR_DQ14"
 		(at 184.15 528.32 0)
@@
 		)
 	)
+	(label "PA10"
+		(at 82.55 146.05 180)
+		(effects
+			(font
+				(size 1.27 1.27)
+			)
+			(justify right bottom)
+		)
+	)
 	(label "PC2"
 		(at 147.32 363.22 180)
@@
 		)
 	)
+	(label "PB15"
+		(at 82.55 72.39 180)
+		(effects
+			(font
+				(size 1.27 1.27)
+			)
+			(justify right bottom)
+		)
+	)
 	(label "USB_HS_D+"
 		(at 314.96 66.04 0)
@@
 		)
 	)
-	(label "PD7"
-		(at 173.99 77.47 0)
-		(effects
-			(font
-				(size 1.27 1.27)
-			)
-			(justify left bottom)
-		)
-	)
 	(label "DDR_DQ8"
 		(at 184.15 510.54 0)
@@
 		)
 	)
+	(label "PB15"
+		(at 43.18 439.42 0)
+		(effects
+			(font
+				(size 1.27 1.27)
+			)
+			(justify left bottom)
+		)
+	)
 	(label "PB7"
 		(at 43.18 419.1 0)
@@
 	)
 	(label "DEBUG0"
-		(at 55.88 408.94 0)
+		(at 26.67 412.75 0)
 		(effects
 			(font
@@
 		)
 	)
+	(label "PA9"
+		(at 43.18 381 0)
+		(effects
+			(font
+				(size 1.27 1.27)
+			)
+			(justify left bottom)
+		)
+	)
 	(label "PG7"
 		(at 173.99 92.71 0)
@@
 	)
 	(label "PG12"
-		(at 167.64 72.39 180)
+		(at 147.32 81.28 180)
 		(effects
 			(font

Commit message: mp133: routing and pin assignment
Connections:
- net PC7 is gone; now on net DEBUG1: U2.C13 (PC7)
- net PG0 is gone; now on net DFU_BOOT: U2.A7 (PG0)
- net PG4 is gone; now on net DEBUG2: U2.B10 (PG4)
- net UART_TX is gone; now on net UART7_TX: J4.1 (Pin_1)
- net DEBUG0: now also U2.B13 (PB5)
- net DEBUG1: no longer U2.C16 (PB4), U2.W10 (PE5)
- net DEBUG3: now also U2.A16 (PF0)
- net PA11: now also J1.55 (Pin_55), J1.56 (Pin_56)
- net PD3: now also J1.41 (Pin_41), J1.42 (Pin_42)
- net PD7: now also J2.71 (Pin_71), J2.72 (Pin_72)
- net PE12: now also J2.1 (Pin_1), J2.2 (Pin_2)
- net PE13: now also J2.17 (Pin_17), J2.18 (Pin_18)
- net PG12: now also J2.75 (Pin_75), J2.76 (Pin_76)
- net PG2: now also J2.69 (Pin_69), J2.70 (Pin_70)
- net PH14: now reaches U2.B8 (PH14)
- net PH14: now also J2.7 (Pin_7), J2.8 (Pin_8)
- net UART7_TX: now reaches U2.E2 (PH2)
- net PB6: now reaches J2.13 (Pin_13), J2.14 (Pin_14)
- net PB6: now also U2.C1 (PB6)
- net PD14: now reaches J2.3 (Pin_3), J2.4 (Pin_4)
- net PD14: now also U2.C4 (PD14)
- net PB4: now reaches J1.1 (Pin_1), J1.2 (Pin_2)
- net PB4: now also U2.C16 (PB4)
- net PB14: now reaches J1.39 (Pin_39), J1.40 (Pin_40)
- net PB14: now also U2.B16 (PB14)
- net PE5: now reaches J1.57 (Pin_57), J1.58 (Pin_58)
- net PE5: now also U2.W10 (PE5)
- net UART7_RX: now reaches U2.C14 (PB3)
- net UART7_RX: now also J4.3 (Pin_3)
- net UART_RX: no longer names the net of U2.B4 (PA15)
- net UART_RX: no longer J4.3 (Pin_3)
Other:
- note added: "I2C5_SCL"
- note added: "I2C5_SDA"
- note removed: "I2C-SCL(withB18)"
- note removed: "I2C-SDA (with A55)"
- note removed: "I2C4_SCL"
- note removed: "I2C4_SDA"
- note removed: "No ADC pin with MOSI and SAI_SD"
- note removed: "No ADC pin with NSS and SAI_FS"
- note removed: "SAI1_MCLK_A"
- note removed: "SAI2_FS"
- note removed: "SAI2_MCLK"
- note removed: "SAI2_SCK"
- note removed: "SAI4_FS_A"
- note removed: "SAI4_MCLK_A"
- note removed: "SAI4_SCK_A"
- note removed: "SAI4_SD_A"
- note removed: "SPI2-MISO"
- note removed: "SPI2-MOSI"
- note removed: "SPI2-NSS"
- note removed: "SPI2_MOSI"
- note removed: "SPI2_NSS"
- note removed: "SPI2_SCK"
- note removed: "SPI3_MISO"
- note removed: "SPI3_SCK"
- note removed: "TIM PWM"
- note removed: "These probably aren't useful bec. other SAI pins don't match mp153-v0.2"
- note removed: "UART_RX"
- note removed: "UART_RX, I2C_SCL"
- note removed: "UART_TX"
- note removed: "nothing (TIM?)"
- note removed: "nothing (codec reset)"

Commit message: mp133: completed routing
Parts:
- added D1: BAT54LP, 4ms_Diode:DFN-1006-2, symbol 4ms_Diode:BAT54LP
- added R6: 10k_0402, 4ms_Resistor:R_0402, symbol 4ms_Resistor_0402:10k_0402
- U21: JLCPCB ID (none) -> C1880992; Part Number AP62301Z6 -> AP62301Z6-7; Part Number 2 AP62300Z6 -> AP62300Z6-7; Part Number 3 AP62300TZ6 -> AP62300TZ6-7
- X2: JLCPCB ID (none) -> C1986107
Connections:
- net NRST: now also D1.1 (K)
- net PWR_ON: now also R6.1
- net PWR_ONRST: no longer U16.5 (EN)
- net  PH11: no longer names the net of U2.K3 (PH11)
- net PA12: no longer names the net of U2.F4 (PA12)
- net PA8: no longer names the net of U2.P2 (PA8)
- net PB0: no longer names the net of U2.W8 (PB0)
- net PB10: no longer names the net of U2.E13 (PB10)
- net PB7: no longer names the net of U2.C6 (PB7)
- net PC0: no longer names the net of U2.W5 (PC0)
- net PC6: no longer names the net of U2.B14 (PC6)
- net PD10: no longer names the net of U2.D6 (PD10)
- net PD11: no longer names the net of U2.F3 (PD11)
- net PD13: no longer names the net of U2.J2 (PD13)
- net PE0: no longer names the net of U2.B6 (PE0)
- net PE10: no longer names the net of U2.C10 (PE10)
- net PE2: no longer names the net of U2.N1 (PE2)
- net PE3: no longer names the net of U2.B17 (PE3)
- net PE4: no longer names the net of U2.H2 (PE4)
- net PE6: no longer names the net of U2.T2 (PE6)
- net PF13: no longer names the net of U2.W4 (PF13)
- net PG1: no longer names the net of U2.R1 (PG1)
- net PG15: no longer names the net of U2.H4 (PG15)
- net PG3: no longer names the net of U2.W1 (PG3)
- net PG5: no longer names the net of U2.G3 (PG5)
- net PG6: no longer names the net of U2.C17 (PG6)
- net PG9: no longer names the net of U2.F2 (PG9)
- net PH6: no longer names the net of U2.N3 (PH6)
- net USB2_DN: no longer names the net of U2.Y13 (USB_DM2)
- net USB2_DP: no longer names the net of U2.AA13 (USB_DP2)
- new net PWR_ONRST2: D1.2 (A), R6.2, U16.5 (EN)
- no-connect marks 23 -> 75
Other:
- note removed: "ADC-0"
- note removed: "ADC-11"
- note removed: "ADC-9"
- note removed: "Bit swapping"
- note removed: "Run these to a header? Jumper to sel?"
- note removed: "SAI2_FS_A"
- note removed: "SAI2_MCLK_A"
- note removed: "SAI2_SD_A"
- note removed: "SAI2_SD_B"
- note removed: "SPI2-SCK"

Commit message: mp133: cleanup for production
Other:
- note added: "SPI4_MOSI"
Changed lines of the file:
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@@
 		)
 	)
-	(text "ADC-2"
+	(text "ADC2-2"
 		(exclude_from_sim no)
 		(at 130.81 360.426 0)
@@
 	(text "ADC-8"
 		(exclude_from_sim no)
-		(at 202.692 419.1 0)
+		(at 206.502 419.1 0)
 		(effects
 			(font
@@
 	(text "ADC-5"
 		(exclude_from_sim no)
-		(at 202.692 421.64 0)
+		(at 206.502 421.64 0)
 		(effects
 			(font
@@
 		)
 	)
+	(text "SPI4_MOSI"
+		(exclude_from_sim no)
+		(at 75.946 72.39 0)
+		(effects
+			(font
+				(size 1.27 1.27)
+			)
+			(justify right bottom)
+		)
+	)
 	(text "SPI3-SCK"
 		(exclude_from_sim no)
@@
 		)
 	)
-	(text "SPI3_MOSI"
+	(text "SPI4_MOSI"
 		(exclude_from_sim no)
 		(at 49.53 439.42 0)
@@
 		)
 	)
-	(text "SPI3_MOSI"
-		(exclude_from_sim no)
-		(at 76.2 72.39 0)
-		(effects
-			(font
-				(size 1.27 1.27)
-			)
-			(justify right bottom)
-		)
-	)
 	(text "          BOOT0  BOOT2\nSD Card    On     On\nFlash      On    Off\nDebugger   Off    On"
 		(exclude_from_sim no)
@@
 	(wire
 		(pts
-			(xy 217.17 411.48) (xy 228.6 411.48)
+			(xy 200.66 411.48) (xy 228.6 411.48)
 		)
 		(stroke
@@
 	(wire
 		(pts
-			(xy 271.78 441.96) (xy 283.21 441.96)
+			(xy 271.78 441.96) (xy 299.72 441.96)
 		)
 		(stroke
@@
 	(wire
 		(pts
-			(xy 271.78 408.94) (xy 283.21 408.94)
+			(xy 271.78 408.94) (xy 299.72 408.94)
 		)
 		(stroke
@@
 	(wire
 		(pts
-			(xy 283.21 358.14) (xy 271.78 358.14)
+			(xy 299.72 358.14) (xy 271.78 358.14)
 		)
 		(stroke
@@
 	(wire
 		(pts
-			(xy 55.88 414.02) (xy 69.85 414.02)
+			(xy 43.18 414.02) (xy 69.85 414.02)
 		)
 		(stroke
@@
 	(wire
 		(pts
-			(xy 196.85 419.1) (xy 228.6 419.1)
+			(xy 200.66 419.1) (xy 228.6 419.1)
 		)
 		(stroke
@@
 	(wire
 		(pts
-			(xy 217.17 406.4) (xy 228.6 406.4)
+			(xy 200.66 406.4) (xy 228.6 406.4)
 		)
 		(stroke
@@
 	(wire
 		(pts
-			(xy 271.78 447.04) (xy 283.21 447.04)
+			(xy 271.78 447.04) (xy 299.72 447.04)
 		)
 		(stroke
@@
 	(wire
 		(pts
-			(xy 217.17 414.02) (xy 228.6 414.02)
+			(xy 200.66 414.02) (xy 228.6 414.02)
 		)
 		(stroke
@@
 	(wire
 		(pts
-			(xy 196.85 421.64) (xy 228.6 421.64)
+			(xy 200.66 421.64) (xy 228.6 421.64)
 		)
 		(stroke
@@
 	(wire
 		(pts
-			(xy 113.03 375.92) (xy 135.89 375.92)
+			(xy 113.03 375.92) (xy 147.32 375.92)
 		)
 		(stroke
@@
 	(wire
 		(pts
-			(xy 271.78 444.5) (xy 289.56 444.5)
+			(xy 271.78 444.5) (xy 303.53 444.5)
 		)
 		(stroke
@@
 	(wire
 		(pts
-			(xy 215.9 426.72) (xy 228.6 426.72)
+			(xy 200.66 426.72) (xy 228.6 426.72)
 		)
 		(stroke
@@
 	(wire
 		(pts
-			(xy 271.78 403.86) (xy 283.21 403.86)
+			(xy 271.78 403.86) (xy 299.72 403.86)
 		)
 		(stroke
@@
 	(wire
 		(pts
-			(xy 271.78 449.58) (xy 283.21 449.58)
+			(xy 271.78 449.58) (xy 299.72 449.58)
 		)
 		(stroke
@@
 	(wire
 		(pts
-			(xy 55.88 406.4) (xy 69.85 406.4)
+			(xy 43.18 406.4) (xy 69.85 406.4)
 		)
 		(stroke
@@
 	(wire
 		(pts
-			(xy 215.9 429.26) (xy 228.6 429.26)
+			(xy 200.66 429.26) (xy 228.6 429.26)
 		)
 		(stroke
@@
 	(wire
 		(pts
-			(xy 217.17 391.16) (xy 228.6 391.16)
+			(xy 200.66 391.16) (xy 228.6 391.16)
 		)
 		(stroke
@@
 	(wire
 		(pts
-			(xy 271.78 401.32) (xy 283.21 401.32)
+			(xy 271.78 401.32) (xy 299.72 401.32)
 		)
 		(stroke
@@
 	(wire
 		(pts
-			(xy 217.17 416.56) (xy 228.6 416.56)
+			(xy 200.66 416.56) (xy 228.6 416.56)
 		)
 		(stroke
@@
 	)
 	(label "JTMS_SWDIO"
-		(at 215.9 429.26 0)
+		(at 200.66 429.26 0)
 		(effects
 			(font
@@
 	)
 	(label "BOOT2"
-		(at 283.21 447.04 180)
+		(at 299.72 447.04 180)
 		(effects
 			(font
@@
 	)
 	(label "DEBUG2"
-		(at 283.21 358.14 180)
+		(at 299.72 358.14 180)
 		(effects
 			(font
@@
 	)
 	(label "FLASH_IO0"
-		(at 217.17 411.48 0)
+		(at 200.66 411.48 0)
 		(effects
 			(font
@@
 	)
 	(label "PF11"
-		(at 196.85 419.1 0)
+		(at 200.66 419.1 0)
 		(effects
 			(font
@@
 	)
 	(label "PF12"
-		(at 196.85 421.64 0)
+		(at 200.66 421.64 0)
 		(effects
 			(font
@@
 	)
 	(label "FLASH_CLK"
-		(at 217.17 416.56 0)
+		(at 200.66 416.56 0)
 		(effects
 			(font
@@
 	)
 	(label "JTDI"
-		(at 283.21 401.32 180)
+		(at 299.72 401.32 180)
 		(effects
 			(font
@@
 	)
 	(label "JTCK_SWCLK"
-		(at 215.9 426.72 0)
+		(at 200.66 426.72 0)
 		(effects
 			(font
@@
 	)
 	(label "JTDO_SWO"
-		(at 283.21 403.86 180)
+		(at 299.72 403.86 180)
 		(effects
 			(font
@@
 	)
 	(label "FLASH_IO1"
-		(at 217.17 414.02 0)
+		(at 200.66 414.02 0)
 		(effects
 			(font
@@
 	)
 	(label "FLASH_IO3"
-		(at 283.21 408.94 180)
+		(at 299.72 408.94 180)
 		(effects
 			(font
@@
 	)
 	(label "DEBUG0"
-		(at 55.88 414.02 0)
+		(at 43.18 414.02 0)
 		(effects
 			(font
@@
 	)
 	(label "DEBUG1"
-		(at 135.89 375.92 180)
+		(at 147.32 375.92 180)
 		(effects
 			(font
@@
 	)
 	(label "DEBUG3"
-		(at 217.17 391.16 0)
+		(at 200.66 391.16 0)
 		(effects
 			(font
@@
 	)
 	(label "USB_VBUS"
-		(at 283.21 449.58 180)
+		(at 299.72 449.58 180)
 		(effects
 			(font
@@
 	)
 	(label "FLASH_CS"
-		(at 55.88 406.4 0)
+		(at 43.18 406.4 0)
 		(effects
 			(font
@@
 	)
 	(label "BOOT0"
-		(at 283.21 441.96 180)
+		(at 299.72 441.96 180)
 		(effects
 			(font
@@
 	)
 	(label "FLASH_IO2"
-		(at 217.17 406.4 0)
+		(at 200.66 406.4 0)
 		(effects
 			(font
@@
 	(symbol
 		(lib_id "4ms_Power_Symbol:GND")
-		(at 289.56 444.5 0)
+		(at 303.53 444.5 0)
 		(mirror y)
 		(unit 1)
@@
 		(fields_autoplaced yes)
 		(property "Reference" "#PWR0110"
-			(at 289.56 450.85 0)
+			(at 303.53 450.85 0)
 			(effects
 				(font
@@
 		)
 		(property "Value" "GND"
-			(at 289.56 448.31 0)
+			(at 303.53 448.31 0)
 			(effects
 				(font
@@
 		)
 		(property "Footprint" ""
-			(at 289.56 444.5 0)
+			(at 303.53 444.5 0)
 			(effects
 				(font
@@
 		)
 		(property "Datasheet" ""
-			(at 289.56 444.5 0)
+			(at 303.53 444.5 0)
 			(effects
 				(font
@@
 		)
 		(property "Description" ""
-			(at 289.56 444.5 0)
+			(at 303.53 444.5 0)
 			(effects
 				(font
