File: sdprog/sdprog/sdprog.kicad_pcb (KiCad board)
At the start: 2 copper layers, 23.7 x 14.6 mm, 10 parts, among them CON1 microSDCon_SMT_104031-0811, J1 Socket_02x05_P1.27mm_SMT

Commit message: Cleanup sdprog
Parts:
- moved C0 2.61 mm to (43.8, 38.4)
- moved D2 2.09 mm to (41.6, 38.4)
- renumbered V0 to C0, B0 to C1
Connections:
- net /BOOT2 renamed /CD1
- net VDD renamed /CD0
Routing:
- net /CD0: track 8.36 -> 10.6 mm
