File: sdprog/sdprog/sdprog.kicad_sch (KiCad schematic)
At the start: 10 parts, among them CON1 microSDCon_SMT_104031-0811, J1 Socket_02x05_P1.27mm_SMT

Commit message: Cleanup sdprog
Connections:
- net BOOT2 renamed CD1
- net VDD renamed CD0
Other:
- note added: "SD card => 1.27mm adaptor"
- moved on the sheet: B0, CK0, D1, D2, D3, V0
