File: mp257/v0.1/mp257-devboard.kicad_sch (KiCad schematic)
At the start: 40 parts, among them CON1 microSDCon_SMT_104031-0811, J1 Pins_02x40_P0.4mm_W3.0mm_SMT, J2 Pins_02x40_P0.4mm_W3.0mm_SMT, J3 USB-C_Receptacle_Molex_217179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, J4 Pins_02x04_RightAngle_P2.54mm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, J5 Conn_01x02, J6 Pins_02x05_P1.27mm_SMT, J7 Conn_02x15_Odd_Even, U1 STM32MP257FAK3, U3 USBLC6-2SC6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

Commit message: Header B almost fully routed
Connections:
- net ADC1_CH10: now also J2.10 (Pin_10), J2.9 (Pin_9)
- net ADC1_CH13: now also J2.47 (Pin_47), J2.48 (Pin_48)
- net ADC1_CH15: now also J2.41 (Pin_41), J2.42 (Pin_42)
- net ADC1_CH16: now also J2.51 (Pin_51), J2.52 (Pin_52)
- net ADC1_CH17: now also J2.39 (Pin_39), J2.40 (Pin_40)
- net ADC1_CH2: now also J2.35 (Pin_35), J2.36 (Pin_36)
- net ADC1_CH4: now also J2.33 (Pin_33), J2.34 (Pin_34)
- net ADC1_CH7: now also J2.43 (Pin_43), J2.44 (Pin_44)
- net ADC3_CH2: now also J2.31 (Pin_31), J2.32 (Pin_32)
- net ADC3_CH4: now also J2.49 (Pin_49), J2.50 (Pin_50)
- net ADC3_CH6: now also J2.29 (Pin_29), J2.30 (Pin_30)
- net ADC3_CH9: now also J2.45 (Pin_45), J2.46 (Pin_46)
- net JTCK_SWCLK: now also U1.AA5 (JTCK_SWCLK)
- net JTDI: now also U1.AE3 (JTDI)
- net JTDO_SWO: now also U1.AC2 (JTDO_SWDO)
- net JTMS_SWDIO: now also U1.AE2 (JTMS_SWDIO)
- net JTRST: now also U1.AF3 (NJTRST)
- net PA10: now also J2.71 (Pin_71), J2.72 (Pin_72), U1.AE15 (PA10)
- net PA9: now also J2.69 (Pin_69), J2.70 (Pin_70); no longer J2.71 (Pin_71), J2.72 (Pin_72)
- net PC4: now also J2.21 (Pin_21), J2.22 (Pin_22), U1.AC9 (PC4)
- net PC8: now reaches J2.11 (Pin_11), J2.12 (Pin_12)
- net PC8: now also U1.AG9 (PC8)
- net PA12: now reaches J2.15 (Pin_15), J2.16 (Pin_16)
- net PA12: now also U1.AC13 (PA12)
- net PF5: now reaches J2.19 (Pin_19), J2.20 (Pin_20)
- net PF5: now also U1.AA11 (PF5)
- no-connect marks 77 -> 72
Other:
- note added: "SAI2_MCLK_B"
- note added: "SPI6_MISO"
- note added: "SPI6_MOSI"
- note added: "SPI6_NSS"
- note added: "SPI6_SCK"

Commit message: Routing...
Connections:
- net FLASH_CLK: now also U1.B17 (PD0)
- net FLASH_CS: now also U1.G13 (PD3)
- net FLASH_IO0: now also U1.C18 (PD4)
- net FLASH_IO1: now also U1.B18 (PD5)
- net FLASH_IO2: now also U1.A18 (PD6)
- net FLASH_IO3: now also U1.D20 (PD7)
- net GND: now also J7.13 (Pin_13), J7.15 (Pin_15); no longer J6.3 (Pin_3), J6.5 (Pin_5), J6.9 (Pin_9), J7.1 (Pin_1), J7.3 (Pin_3), J7.5 (Pin_5), J7.7 (Pin_7), J7.9 (Pin_9)
- net JTCK_SWCLK: no longer J6.4 (Pin_4)
- net JTDI: no longer J6.8 (Pin_8)
- net JTDO_SWO: no longer J6.6 (Pin_6)
- net JTMS_SWDIO: no longer J6.2 (Pin_2)
- net PB4: now also J1.57 (Pin_57), J1.58 (Pin_58), U1.B15 (PB4)
- net PB6: now also J2.5 (Pin_5), J2.6 (Pin_6); no longer J1.3 (Pin_3), J1.4 (Pin_4)
- net PD2: now also J1.41 (Pin_41), J1.42 (Pin_42), U1.D12 (PD2)
- net PE9: no longer J1.41 (Pin_41), J1.42 (Pin_42)
- net PH7: now also J1.3 (Pin_3), J1.4 (Pin_4); no longer J2.5 (Pin_5), J2.6 (Pin_6)
- net VDD: no longer J6.1 (Pin_1)
- net LTDC_R1: now reaches J7.11 (Pin_11)
- net LTDC_R1: now also U1.AB8 (PF7)
- net LTDC_G0: now reaches J7.17 (Pin_17)
- net LTDC_G0: now also U1.AE10 (PF8)
- net LTDC_R2: now reaches J7.19 (Pin_19)
- net LTDC_R2: now also U1.P2 (PF13)
- net LTDC_B0: now reaches U1.U1 (PI9)
- net LTDC_B0: now also J7.9 (Pin_9)
- net PB0: now reaches J1.1 (Pin_1), J1.2 (Pin_2)
- net PB0: now also U1.B13 (PB0)
- net PB2: now reaches J1.5 (Pin_5), J1.6 (Pin_6)
- net PB5: now reaches J1.55 (Pin_55), J1.56 (Pin_56)
- net PB5: now also U1.C14 (PB5)
- net at J6.10 (Pin_10): no longer JP1.2 (C)
- net LTDC_R0: now reaches U1.AB16 (PH4)
- net LTDC_R0: now also J7.1 (Pin_1)
- net LTDC_G1: now reaches U1.AG18 (PH5)
- net LTDC_G1: now also J7.3 (Pin_3)
- net LTDC_B2: now reaches U1.K6 (PG15)
- net LTDC_B2: now also J7.7 (Pin_7)
- net LTDC_B1: now reaches U1.N1 (PG14)
- net LTDC_B1: now also J7.5 (Pin_5)
- no-connect marks 72 -> 68
Other:
- note added: "I2C2_SCL"
- note added: "I2C2_SDA"
- note added: "SPI1_MOSI"
- note added: "SPI1_NSS"
- note added: "SPI1_SCK"
- note added: "SPI2_MOSI"
- note added: "SPI2_SCK"
- note added: "UART4_TX(swapRX)"
- note removed: "ADC-1"
- note removed: "ADC-10"
- note removed: "ADC-12"
- note removed: "ADC-13"
- note removed: "ADC-14"
- note removed: "ADC-15"
- note removed: "ADC-16"
- note removed: "ADC-17"
- note removed: "ADC-2"
- note removed: "ADC-3"
- note removed: "ADC-4"
- note removed: "ADC-5"
- note removed: "ADC-6"
- note removed: "ADC-7"
- note removed: "ADC-8"
- note removed: "ADC2-2"
- note removed: "I2C1_SCL"
- note removed: "I2C1_SDA"
- note removed: "I2C3_SCL"
- note removed: "I2C3_SDA"
- note removed: "I2C5_SCL"
- note removed: "SAI1_FS"
- note removed: "SAI1_MCLK"
- note removed: "SAI1_SCK"
- note removed: "SAI1_SD_A"
- note removed: "SAI1_SD_B"
- note removed: "SAI2_SCK_A"
- note removed: "SDMMC_CMD"
- note removed: "SPI3-MISO"
- note removed: "SPI3-SCK"
- note removed: "SPI3_MOSI"
- note removed: "SPI3_NSS"
- note removed: "SPI4_MOSI"
- note removed: "TIM1_CH3"
- note removed: "UART4_TX"
- moved on the sheet: J6

Commit message: Routing
Connections:
- net GND: now also J6.3 (Pin_3), J6.5 (Pin_5), J6.9 (Pin_9)
- net JTCK_SWCLK: now also J6.4 (Pin_4)
- net JTDI: now also J6.8 (Pin_8)
- net JTDO_SWO: now also J6.6 (Pin_6)
- net JTMS_SWDIO: now also J6.2 (Pin_2)
- net PB2: now also U1.A14 (PB2)
- net VDD: now also J6.1 (Pin_1)
- net at J6.10 (Pin_10): now also JP1.2 (C)
Other:
- moved on the sheet: J6
Changed lines of the file:
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@@
 		)
 	)
+	(text "SPI2_MOSI"
+		(exclude_from_sim no)
+		(at 51.308 384.302 0)
+		(effects
+			(font
+				(size 1.27 1.27)
+			)
+			(justify right bottom)
+		)
+	)
 	(text "SPI1_NSS"
 		(exclude_from_sim no)
@@
 	)
 	(junction
+		(at 49.53 199.39)
+		(diameter 0)
+		(color 0 0 0 0)
+	)
+	(junction
 		(at 160.02 118.11)
 		(diameter 0)
@@
 	(wire
 		(pts
+			(xy 36.83 384.81) (xy 62.23 384.81)
+		)
+		(stroke
+			(width 0)
+			(type default)
+		)
+	)
+	(wire
+		(pts
 			(xy 49.53 96.52) (xy 49.53 99.06)
 		)
@@
 		)
 	)
+	(label "PB2"
+		(at 36.83 384.81 0)
+		(effects
+			(font
+				(size 1.27 1.27)
+			)
+			(justify left bottom)
+		)
+	)
 	(label "LTDC_VSYNC"
 		(at 243.84 134.62 180)
@@
 	(symbol
 		(lib_id "4ms_Connector:Pins_02x05_P1.27mm_SMT")
-		(at 55.88 201.93 90)
+		(at 55.88 201.93 0)
 		(unit 1)
 		(exclude_from_sim no)
@@
 		(dnp no)
 		(property "Reference" "J6"
-			(at 45.72 201.93 0)
+			(at 55.88 191.77 0)
 			(effects
 				(font
@@
 		)
 		(property "Value" "Pins_02x05_P1.27mm_SMT"
-			(at 63.5 201.93 0)
+			(at 55.88 209.55 0)
 			(effects
 				(font
@@
 		)
 		(property "Footprint" "4ms_Connector:Pins_2x05_1.27mm_SMD"
-			(at 72.39 200.025 0)
+			(at 57.785 218.44 0)
 			(effects
 				(font
@@
 		)
 		(property "Datasheet" "https://www.mouser.com/datasheet/2/527/ftsh_smt-1316912.pdf"
-			(at 55.88 203.2 0)
+			(at 54.61 201.93 0)
 			(effects
 				(font
@@
 		)
 		(property "Specifications" "Header 2x5 Pins, Pitch=1.27mm, Pin Height=3mm, Vertical, SMT"
-			(at 66.675 200.66 0)
+			(at 57.15 212.725 0)
 			(effects
 				(font
@@
 		)
 		(property "Manufacturer" "Samtec"
-			(at 68.58 202.565 0)
+			(at 55.245 214.63 0)
 			(effects
 				(font
@@
 		)
 		(property "Part Number" "FTSH-105-01-F-DV"
-			(at 70.485 203.2 0)
+			(at 54.61 216.535 0)
 			(effects
 				(font

Commit message: Routing: moved chips closer to B header
Parts:
- added R13, R14: 200Ω_0402, 4ms_Resistor:R_0402, symbol 4ms_Resistor_0402:200Ω_0402
Connections:
- net GND: now also R13.2, R14.2
- net PE9: now also J1.39 (Pin_39), J1.40 (Pin_40)
- net USB3_DM: no longer U1.AF22 (USB3DR_DP)
- net USB_HS_DM: no longer U1.AG21 (USBH_HS_DM)
- net USB_VBUS: now also U1.AE19 (PH3)
- net LVDS1_D0P: now reaches U1.G2 (LVDS1_D0P)
- net LVDS1_D0N: now reaches U1.G3 (LVDS1_D0N)
- net LVDS1_D1P: now reaches U1.H3 (LVDS1_D1P)
- net LVDS1_D1N: now reaches U1.H4 (LVDS1_D1N)
- net LVDS1_D2P: now reaches U1.J1 (LVDS1_D2P)
- net LVDS1_D2N: now reaches U1.J2 (LVDS1_D2N)
- net LVDS1_D4P: now reaches U1.K1 (LVDS1_D4P)
- net LVDS1_D4N: now reaches U1.K2 (LVDS1_D4N)
- net LVDS1_D3P: now reaches U1.L2 (LVDS1_D3P)
- net LVDS1_D3N: now reaches U1.L3 (LVDS1_D3N)
- net DSI_D1N: now reaches U1.A10 (DSI_D1N)
- net DSI_D3P: now reaches U1.A6 (DSI_D3P)
- net DSI_D2N: now reaches U1.A7 (DSI_D2N)
- net DSI_D1P: now reaches U1.B10 (DSI_D1P)
- net DSI_D3N: now reaches U1.B6 (DSI_D3N)
- net DSI_D2P: now reaches U1.B7 (DSI_D2P)
- net DSI_D0P: now reaches U1.B9 (DSI_D0P)
- net DSI_CKP: now reaches U1.C7 (DSI_CKP)
- net DSI_CKN: now reaches U1.C8 (DSI_CKN)
- net DSI_D0N: now reaches U1.C9 (DSI_D0N)
- net at U1.D6 (DSI_REXT): now also R14.1
- net PH8: now reaches J2.3 (Pin_3), J2.4 (Pin_4)
- net PH8: now also U1.AD16 (PH8)
- net PD13: now reaches J1.63 (Pin_63), J1.64 (Pin_64)
- net PD13: now also U1.D25 (PD13)
- net at U1.AF23 (USB3DR_TXRTUNE): now also R13.1
- new net USB3_DN: U1.AF22 (USB3DR_DP)
- new net USB_HS_DN: U1.AG21 (USBH_HS_DM)
- no-connect marks 68 -> 46
Other:
- moved on the sheet: U1D, U1I

Commit message: WIP routing
Parts:
- removed R3, R6, R7, R8: 0Ω_0603, 4ms_Resistor:R_0603, symbol 4ms_Resistor_0603:0Ω_0603
- added R15, R16, R17: 10k_0402, 4ms_Resistor:R_0402, symbol 4ms_Resistor_0402:10k_0402
- added SJ1: Jumper, 4ms_SolderJumper:JUMPER_SMD_1x2, symbol 4ms_Net_Tie:Jumper-Open
Connections:
- net BOOT0: now also R15.1
- net BOOT2: now also R17.1
- net GND: now also R15.2, R16.2, R17.2
- net USB3_DN: now also U3.3 (I/O2)
- net USB3_DP: now also U3.1 (I/O1)
- net VDD: now also SJ1.2 (B)
- net LVDS1_D0N: no longer names the net of U1.G3 (LVDS1_D0N)
- net LVDS1_D0P: no longer names the net of U1.G2 (LVDS1_D0P)
- net LVDS1_D1N: no longer names the net of U1.H4 (LVDS1_D1N)
- net LVDS1_D1P: no longer names the net of U1.H3 (LVDS1_D1P)
- net LVDS1_D2N: no longer names the net of U1.J2 (LVDS1_D2N)
- net LVDS1_D2P: no longer names the net of U1.J1 (LVDS1_D2P)
- net LVDS1_D3N: no longer names the net of U1.L3 (LVDS1_D3N)
- net LVDS1_D3P: no longer names the net of U1.L2 (LVDS1_D3P)
- net LVDS1_D4N: no longer names the net of U1.K2 (LVDS1_D4N)
- net LVDS1_D4P: no longer names the net of U1.K1 (LVDS1_D4P)
- new net BOOT1: R16.1, SJ1.1 (A)
- no-connect marks 46 -> 56
Other:
- note added: "BOOT0 BOOT1 BOOT2 SD Card On Off Off Flash Off Off On Debugger On On Off"
- note removed: "BOOT0 BOOT2 SD Card On On Flash On Off Debugger Off On"
- moved on the sheet: R72

Commit message: Routing WIP
Parts:
- removed J7: Conn_02x15_Odd_Even, 4ms_Connector:Connector-30pin-P0.4mm-W3.0mm, symbol Connector_Generic:Conn_02x15_Odd_Even
- added J7: Conn_02x20_Odd_Even, 4ms_Connector:Connector-40pin-P0.4mm-W3.0mm, symbol Connector_Generic:Conn_02x20_Odd_Even
Connections:
- net GND: now also J7.23 (Pin_23), J7.25 (Pin_25)
- net LTDC_B0: now also J7.19 (Pin_19)
- net LTDC_B1: now also J7.15 (Pin_15)
- net LTDC_B2: now also J7.17 (Pin_17)
- net LTDC_B3: now also J7.33 (Pin_33)
- net LTDC_B4: now also J7.31 (Pin_31)
- net LTDC_B5: now also J7.20 (Pin_20)
- net LTDC_B6: now also J7.18 (Pin_18)
- net LTDC_B7: now also J7.16 (Pin_16)
- net LTDC_CLK: now also J7.35 (Pin_35)
- net LTDC_DE: now also J7.14 (Pin_14)
- net LTDC_G0: now also J7.27 (Pin_27)
- net LTDC_G1: now also J7.13 (Pin_13)
- net LTDC_G2: now also J7.30 (Pin_30)
- net LTDC_G3: now also J7.32 (Pin_32)
- net LTDC_G4: now also J7.34 (Pin_34)
- net LTDC_G5: now also J7.36 (Pin_36)
- net LTDC_G6: now also J7.38 (Pin_38)
- net LTDC_G7: now also J7.40 (Pin_40)
- net LTDC_HSYNC: now also J7.22 (Pin_22)
- net LTDC_R0: now also J7.11 (Pin_11)
- net LTDC_R1: now also J7.21 (Pin_21)
- net LTDC_R2: now also J7.29 (Pin_29)
- net LTDC_R3: now also J7.37 (Pin_37)
- net LTDC_R4: now also J7.39 (Pin_39)
- net LTDC_R5: now also J7.24 (Pin_24)
- net LTDC_R6: now also J7.26 (Pin_26)
- net LTDC_R7: now also J7.28 (Pin_28)
- net LTDC_VSYNC: now also J7.12 (Pin_12)
- net USB3_DN: now also J1.77 (Pin_77), J1.78 (Pin_78)
- net USB3_DP: now also J1.75 (Pin_75), J1.76 (Pin_76)
- net USB_HS_D+: no longer J1.75 (Pin_75), J1.76 (Pin_76)
- net USB_HS_D-: no longer J1.77 (Pin_77), J1.78 (Pin_78)
Other:
- moved on the sheet: R14, U1D, U1I

Commit message: routing
Connections:
- net GND: no longer CON1.11 (SDDET2)
- net PB11: now reaches CON1.10 (SDDET1)
- net PB11: now also J1.11 (Pin_11), J1.12 (Pin_12), U1.A11 (PB11)
- net PB10: now reaches U1.B11 (PB10)
- net PB10: now also CON1.11 (SDDET2)
Other:
- note added: "SD_CARD_DETECT2"
Changed lines of the file:
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@@
 	(text "SD_CARD_DETECT"
 		(exclude_from_sim no)
-		(at 204.216 297.18 0)
+		(at 196.088 297.18 0)
 		(effects
 			(font
@@
 		)
 	)
+	(text "SD_CARD_DETECT2"
+		(exclude_from_sim no)
+		(at 196.342 299.466 0)
+		(effects
+			(font
+				(size 1.27 1.27)
+			)
+			(justify left bottom)
+		)
+	)
 	(text "NOR Flash"
 		(exclude_from_sim no)
@@
 	(wire
 		(pts
+			(xy 189.23 299.72) (xy 223.52 299.72)
+		)
+		(stroke
+			(width 0)
+			(type default)
+		)
+	)
+	(wire
+		(pts
 			(xy 49.53 147.32) (xy 82.55 147.32)
 		)
@@
 	(wire
 		(pts
+			(xy 36.83 407.67) (xy 62.23 407.67)
+		)
+		(stroke
+			(width 0)
+			(type default)
+		)
+	)
+	(wire
+		(pts
 			(xy 36.83 458.47) (xy 62.23 458.47)
 		)
@@
 	(wire
 		(pts
+			(xy 36.83 405.13) (xy 62.23 405.13)
+		)
+		(stroke
+			(width 0)
+			(type default)
+		)
+	)
+	(wire
+		(pts
 			(xy 46.99 264.16) (xy 35.56 264.16)
 		)
@@
 	(wire
 		(pts
-			(xy 220.98 299.72) (xy 223.52 299.72)
-		)
-		(stroke
-			(width 0)
-			(type default)
-		)
-	)
-	(wire
-		(pts
 			(xy 300.99 93.98) (xy 300.99 96.52)
 		)
@@
 		)
 	)
+	(label "PB11"
+		(at 36.83 407.67 0)
+		(effects
+			(font
+				(size 1.27 1.27)
+			)
+			(justify left bottom)
+		)
+	)
 	(label "PA9"
 		(at 36.83 356.87 0)
@@
 		)
 	)
+	(label "PB11"
+		(at 82.55 68.58 180)
+		(effects
+			(font
+				(size 1.27 1.27)
+			)
+			(justify right bottom)
+		)
+	)
 	(label "USB_VBUS_JACK"
 		(at 264.16 127 0)
@@
 		)
 	)
+	(label "PB10"
+		(at 36.83 405.13 0)
+		(effects
+			(font
+				(size 1.27 1.27)
+			)
+			(justify left bottom)
+		)
+	)
 	(label "LTDC_G1"
 		(at 250.19 392.43 180)
@@
 		)
 	)
+	(label "PB11"
+		(at 189.23 297.18 0)
+		(effects
+			(font
+				(size 1.27 1.27)
+			)
+			(justify left bottom)
+		)
+	)
 	(label "ADC1_CH12"
 		(at 132.08 130.81 0)
@@
 		)
 	)
+	(label "PB10"
+		(at 189.23 299.72 0)
+		(effects
+			(font
+				(size 1.27 1.27)
+			)
+			(justify left bottom)
+		)
+	)
 	(label "LTDC_B7"
 		(at 36.83 455.93 0)
@@
 					(unit 1)
 				)
-			)
-		)
-	)
-	(symbol
-		(lib_id "power:GND")
-		(at 220.98 299.72 0)
-		(unit 1)
-		(exclude_from_sim no)
-		(in_bom yes)
-		(on_board yes)
-		(dnp no)
-		(property "Reference" "#PWR039"
-			(at 220.98 299.72 0)
-			(effects
-				(font
-					(size 1.27 1.27)
-				)
-				(hide yes)
-			)
-		)
-		(property "Value" "GND"
-			(at 220.98 303.53 0)
-			(effects
-				(font
-					(size 1.27 1.27)
-				)
-			)
-		)
-		(property "Footprint" ""
-			(at 220.98 299.72 0)
-			(effects
-				(font
-					(size 1.27 1.27)
-				)
-				(hide yes)
-			)
-		)
-		(property "Datasheet" ""
-			(at 220.98 299.72 0)
-			(effects
-				(font
-					(size 1.27 1.27)
-				)
-				(hide yes)
-			)
-		)
-		(property "Description" ""
-			(at 220.98 299.72 0)
-			(effects
-				(font
-					(size 1.27 1.27)
-				)
-				(hide yes)
-			)
-		)
-		(pin "1"
-		)
-		(instances
-			(project "mp153-devboard"
-				(path "/64ec1a6b-f4f9-4414-abbd-a05816451f08"
-					(reference "#PWR039")
-					(unit 1)
-				)

Commit message: Routing
Connections:
- net DSI_CKN: now also J7.9 (Pin_9)
- net DSI_CKP: now also J7.11 (Pin_11)
- net DSI_D0N: now also J7.5 (Pin_5)
- net DSI_D0P: now also J7.7 (Pin_7)
- net DSI_D1N: now also J7.3 (Pin_3)
- net DSI_D1P: now also J7.1 (Pin_1)
- net DSI_D2N: now also J7.4 (Pin_4)
- net DSI_D2P: now also J7.2 (Pin_2)
- net DSI_D3N: now also J7.8 (Pin_8)
- net DSI_D3P: now also J7.6 (Pin_6)
- net LTDC_B0: now also J7.38 (Pin_38); no longer J7.19 (Pin_19)
- net LTDC_B1: now also J7.20 (Pin_20); no longer J7.15 (Pin_15)
- net LTDC_B2: now also J7.13 (Pin_13); no longer J7.17 (Pin_17)
- net LTDC_B3: now also J7.19 (Pin_19); no longer J7.33 (Pin_33)
- net LTDC_B4: now also J7.17 (Pin_17); no longer J7.31 (Pin_31)
- net LTDC_B5: now also J7.21 (Pin_21); no longer J7.20 (Pin_20)
- net LTDC_B6: now also J7.29 (Pin_29); no longer J7.18 (Pin_18)
- net LTDC_B7: now also J7.31 (Pin_31); no longer J7.16 (Pin_16)
- net LTDC_CLK: now also J7.28 (Pin_28); no longer J7.35 (Pin_35)
- net LTDC_DE: now also J7.15 (Pin_15); no longer J7.14 (Pin_14)
- net LTDC_G0: now also J7.39 (Pin_39); no longer J7.27 (Pin_27)
- net LTDC_G1: now also J7.33 (Pin_33); no longer J7.13 (Pin_13)
- net LTDC_G2: now also J7.14 (Pin_14); no longer J7.30 (Pin_30)
- net LTDC_G3: now also J7.16 (Pin_16); no longer J7.32 (Pin_32)
- net LTDC_G4: now also J7.18 (Pin_18); no longer J7.34 (Pin_34)
- net LTDC_G5: now also J7.22 (Pin_22); no longer J7.36 (Pin_36)
- net LTDC_G6: now also J7.27 (Pin_27); no longer J7.38 (Pin_38)
- net LTDC_G7: now also J7.24 (Pin_24); no longer J7.40 (Pin_40)
- net LTDC_HSYNC: now also J7.12 (Pin_12); no longer J7.22 (Pin_22)
- net LTDC_R0: now also J7.35 (Pin_35); no longer J7.11 (Pin_11)
- net LTDC_R1: now also J7.37 (Pin_37); no longer J7.21 (Pin_21)
- net LTDC_R2: now also J7.26 (Pin_26); no longer J7.29 (Pin_29)
- net LTDC_R3: now also J7.32 (Pin_32); no longer J7.37 (Pin_37)
- net LTDC_R4: now also J7.30 (Pin_30); no longer J7.39 (Pin_39)
- net LTDC_R5: now also J7.34 (Pin_34); no longer J7.24 (Pin_24)
- net LTDC_R6: now also J7.36 (Pin_36); no longer J7.26 (Pin_26)
- net LTDC_R7: now also J7.40 (Pin_40); no longer J7.28 (Pin_28)
- net LTDC_VSYNC: now also J7.10 (Pin_10); no longer J7.12 (Pin_12)
Other:
- moved on the sheet: J7
