File: mp257/v0.1/mp257-devboard.kicad_sch (KiCad schematic)
At the start: 39 parts, among them CON1 microSDCon_SMT_104031-0811, J1 Pins_02x40_P0.4mm_W3.0mm_SMT, J2 Pins_02x40_P0.4mm_W3.0mm_SMT, J3 USB-C_Receptacle_Molex_217179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, J4 Pins_02x04_RightAngle_P2.54mm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, J5 Conn_01x02, J6 Pins_02x05_P1.27mm_SMT, J7 Conn_02x20_Odd_Even, U1 STM32MP257FAK3, U3 USBLC6-2SC6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

Commit message: Cleanup BOM, update all parts from lib
Parts:
- H1, H2, H3: value Spacer Nylon, fits 3mm hole -> Spacer Nylon, Unthreaded, Height=11mm, ID >= 3mm, OD < 6mm; Manufacturer (none) -> McMaster-Carr; Part Number (none) -> 93657A504; Specifications Spacer Nylon, fits 3mm hole -> Spacer Nylon, Unthreaded, Height=11mm, ID >= 3mm, OD < 6mm
- J5: value Conn_01x02 -> Pins_01x02_RightAngle_P2.54mm_TH; symbol 4ms_Connector:Conn_01x02 -> 4ms_Connector:Pins_01x02_RightAngle_P2.54mm_TH; Specifications Pins_01x02, Header, Male Pins, 1*2, spacing 2.54mm, right a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 -> HEADER 1x2 MALE PINS 0.100” 90deg
- JP1: footprint 4ms_SolderJumper:JUMPER_SMD_1x3_tiny -> 4ms_SolderJumper:JUMPER_SMD_1x3_tiny_shorted12
- U1: ALTIUM_VALUE STM32MP257FAK3 -> (none); COMPONENTLINK1URL http://tunmcdsvn.tun.st.com/Component_Documentation_Library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 -> (none); COMPONENT_COUNTRY_OF_ORIGIN Unknown -> (none); ID 5491 -> (none); INTERNAL_PART_NUMBER MCD-03375 -> (none); MANUFACTURER STMICROELECTRONICS -> (none); MANUFACTURER_PART_NUMBER STM32MP257FAK3 -> (none); Manufacturer (none) -> STMICROELECTRONICS; ORDER_CODE_DIGIKEY N/A -> (none); ORDER_CODE_FARNELL N/A -> (none); ORDER_CODE_RS N/A -> (none); PACKAGE TFBGA -> (none); PART_PREFERENCE Recommended -> (none); PART_TYPE IC -> (none); Part Number (none) -> STM32MP257FAK3; SHOWFIELDS YES -> (none); STATUS Checked -> (none); Specifications (none) -> STM32MP257FAK3 MPU

Commit message: Finish board, cleanup BOM
Parts:
- D1, D2: symbol Diode:ESD5Zxx -> 4ms_Diode:ESD7351XV2T1G; Manufacturer (none) -> onsemi; Manufacturer_1 (none) -> onsemi; Part Number (none) -> ESD7351XV2T1G; Part Number 2 (none) -> ESD5Z3.3T1G
- J7: value Conn_02x20_Odd_Even -> Pins_02x20_P0.4mm_W3.0mm_SMT; symbol Connector_Generic:Conn_02x20_Odd_Even -> 4ms_Connector:Pins_02x20_P0.4mm_W3.0mm_SMT; JLCPCB ID (none) -> C424643; Manufacturer (none) -> Hirose; Part Number (none) -> DF40C-40DP-0.4V(51)
- SJ1: now not fitted; now left out of the parts list
- X2: JLCPCB ID (none) -> C50396645; Manufacturer ECS -> Murata; Manufacturer 2 (none) -> NDK; Part Number (none) -> XRCGB40M000F0G00R0; Part Number 2 (none) -> NX2016SA-40MHZ-STD-CZS-3
Changed lines of the file:
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@@
 	)
 	(symbol
-		(lib_id "Diode:ESD5Zxx")
+		(lib_id "4ms_Diode:ESD7351XV2T1G")
 		(at 321.31 87.63 270)
 		(unit 1)
@@
 			)
 		)
-		(property "Description" "ESD Protection Diode, SOD-523"
+		(property "Description" "ESD Protection Diode, SOD-523, Vrwm=3.3V, Vclamp@1A=8V, C < 150pF"
 			(at 321.31 87.63 0)
 			(effects
@@
 			)
 		)
-		(property "Note" ""
-			(at 321.31 87.63 90)
+		(property "Manufacturer" "onsemi"
+			(at 321.31 87.63 0)
+			(effects
+				(font
+					(size 1.27 1.27)
+				)
+				(hide yes)
+			)
+		)
+		(property "Part Number" "ESD7351XV2T1G "
+			(at 321.31 87.63 0)
+			(effects
+				(font
+					(size 1.27 1.27)
+				)
+				(hide yes)
+			)
+		)
+		(property "Manufacturer_1" "onsemi"
+			(at 321.31 87.63 0)
+			(effects
+				(font
+					(size 1.27 1.27)
+				)
+				(hide yes)
+			)
+		)
+		(property "Part Number 2" "ESD5Z3.3T1G"
+			(at 321.31 87.63 0)
 			(effects
 				(font
@@
 	)
 	(symbol
-		(lib_id "Diode:ESD5Zxx")
+		(lib_id "4ms_Diode:ESD7351XV2T1G")
 		(at 308.61 87.63 270)
 		(unit 1)
@@
 			)
 		)
-		(property "Description" "ESD Protection Diode, SOD-523"
+		(property "Description" "ESD Protection Diode, SOD-523, Vrwm=3.3V, Vclamp@1A=8V, C < 150pF"
 			(at 308.61 87.63 0)
 			(effects
@@
 			)
 		)
-		(property "Note" ""
-			(at 308.61 87.63 90)
+		(property "Manufacturer" "onsemi"
+			(at 308.61 87.63 0)
+			(effects
+				(font
+					(size 1.27 1.27)
+				)
+				(hide yes)
+			)
+		)
+		(property "Part Number" "ESD7351XV2T1G "
+			(at 308.61 87.63 0)
+			(effects
+				(font
+					(size 1.27 1.27)
+				)
+				(hide yes)
+			)
+		)
+		(property "Manufacturer_1" "onsemi"
+			(at 308.61 87.63 0)
+			(effects
+				(font
+					(size 1.27 1.27)
+				)
+				(hide yes)
+			)
+		)
+		(property "Part Number 2" "ESD5Z3.3T1G"
+			(at 308.61 87.63 0)
 			(effects
 				(font
@@
 	)
 	(symbol
-		(lib_id "Connector_Generic:Conn_02x20_Odd_Even")
+		(lib_id "4ms_Connector:Pins_02x20_P0.4mm_W3.0mm_SMT")
 		(at 219.71 154.94 0)
 		(unit 1)
@@
 			)
 		)
-		(property "Value" "Conn_02x20_Odd_Even"
+		(property "Value" "Pins_02x20_P0.4mm_W3.0mm_SMT"
 			(at 220.98 128.27 0)
 			(effects
@@
 			)
 		)
-		(property "Description" "Generic connector, double row, 02x20, odd/even pin numbering scheme (row 1 odd numbers, row 2 even numbers), script generated (kicad-library-utils/schlib/autogen/connector/)"
+		(property "Description" "Hi-speed board to board connector, 2 x 20 pins"
 			(at 219.71 154.94 0)
 			(effects
@@
 			)
 		)
-		(property "Note" ""
+		(property "Manufacturer" "Hirose"
+			(at 219.71 154.94 0)
+			(effects
+				(font
+					(size 1.27 1.27)
+				)
+				(hide yes)
+			)
+		)
+		(property "Part Number" "DF40C-40DP-0.4V(51)"
+			(at 219.71 154.94 0)
+			(effects
+				(font
+					(size 1.27 1.27)
+				)
+				(hide yes)
+			)
+		)
+		(property "JLCPCB ID" "C424643"
 			(at 219.71 154.94 0)
 			(effects
@@
 					(size 1.27 1.27)
 				)
+				(hide yes)
 			)
 		)
@@
 			)
 		)
-		(property "Manufacturer" "ECS"
+		(property "Manufacturer" "Murata"
 			(at 290.83 377.19 0)
 			(effects
@@
 			)
 		)
-		(property "Part Number" ""
+		(property "Part Number" "XRCGB40M000F0G00R0"
 			(at 288.29 378.46 0)
 			(effects
@@
 			)
 		)
-		(property "JLCPCB ID" ""
+		(property "JLCPCB ID" "C50396645"
 			(at 298.45 377.19 0)
 			(effects
@@
 			)
 		)
+		(property "Manufacturer 2" "NDK"
+			(at 278.13 377.19 0)
+			(effects
+				(font
+					(size 1.27 1.27)
+				)
+				(hide yes)
+			)
+		)
+		(property "Part Number 2" "NX2016SA-40MHZ-STD-CZS-3"
+			(at 278.13 377.19 0)
+			(effects
+				(font
+					(size 1.27 1.27)
+				)
+				(hide yes)
+			)
+		)
 		(pin "4"
 		)
@@
 		(on_board yes)
 		(dnp no)
-		(fields_autoplaced yes)
 		(property "Reference" "#PWR034"
 			(at 321.31 102.87 0)
@@
 		)
 		(property "Description" "Power symbol creates a global label with name \"GND\" , ground"
-			(at 321.31 96.52 0)
+			(at 321.818 104.648 0)
 			(effects
 				(font
 					(size 1.27 1.27)
 				)
+				(hide yes)
 			)
 		)
@@
 		(at 358.14 217.17 0)
 		(unit 1)
-		(exclude_from_sim no)
-		(in_bom yes)
+		(exclude_from_sim yes)
+		(in_bom no)
 		(on_board yes)
-		(dnp no)
+		(dnp yes)
 		(property "Reference" "SJ1"
 			(at 358.14 212.09 0)

Commit message: BOOT pin notes
Other:
- note added: "BOOT3 is GND"
- note added: "Boot 0 1 2 (towards USB is 1, towards reset button is 0; boot1 open = 0, blobbed=1) 0 0 0 = 0 forced USB: no sd clk, no flash cs 1 0 0 = 1 A35 SDMMC1: but no sd clk, no flash cs 0 1 0 = 2 A35 eMMC: no pins 1 1 0 = 3 Dev boot: no pins 0 0 1 = 4 A35 QSPI Serial NOR: two neg pulses on flash cs, 32MHz clock on flash clk (60 pulses each) 1 0 1 = 5 not valid??: no sd clk, lots of neg pulses on flash cs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"
