File: mp257/v0.1/mp257-devboard.kicad_sch (KiCad schematic)
At the start: 39 parts, among them CON1 microSDCon_SMT_104031-0811, J1 Pins_02x40_P0.4mm_W3.0mm_SMT, J2 Pins_02x40_P0.4mm_W3.0mm_SMT, J3 USB-C_Receptacle_Molex_217179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, J4 Pins_02x04_RightAngle_P2.54mm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, J5 Pins_01x02_RightAngle_P2.54mm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, J6 Pins_02x05_P1.27mm_SMT, J7 Pins_02x20_P0.4mm_W3.0mm_SMT, U1 STM32MP257FAK3, U3 USBLC6-2SC6, U5 NORFLASH_W25Q128JV, X2 40MHz_6.8pF_2x1.6mm

Commit message: update to kicad10
Other:
- note added: "C"
