File: mp257/v0.1/mp257-devboard.kicad_pcb (KiCad board)
At the start: 4 copper layers, 42.2 x 57.9 mm, 225 parts, among them CON1 microSDCon_SMT_104031-0811, J1 Pins_02x40_P0.4mm_W3.0mm_SMT, J2 Pins_02x40_P0.4mm_W3.0mm_SMT, J3 USB-C_Receptacle_Molex_217179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, J4 Pins_02x04_RightAngle_P2.54mm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, J5 Conn_01x02, J6 Pins_02x05_P1.27mm_SMT, J7 Conn_02x20_Odd_Even, U1 STM32MP257FAK3, U15 MT40A1G16TB-062E IT:F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

Commit message: Cleanup BOM, update all parts from lib
Parts:
- C194: value 10uF_0603_10V -> 10uF_0402_6.3V
- C225, C235: footprint 4ms_Capacitor:C_0201 -> 4ms_Capacitor:C_0201_TightCourtyard
- C234: value 100nF_0201_16V -> 100nF_0402_16V
- H1, H2, H3: value Spacer Nylon, fits 3mm hole -> Spacer Nylon, Unthreaded, Height=11mm, ID >= 3mm, OD < 6mm
- J5: value Conn_01x02 -> Pins_01x02_RightAngle_P2.54mm_TH
- JP1: footprint 4ms_SolderJumper:JUMPER_SMD_1x3_tiny -> 4ms_SolderJumper:JUMPER_SMD_1x3_tiny_shorted12
- R11: value 0Ω_0603 -> 0Ω_0402
- R174: value 240Ω_0402 -> 240Ω_0201
