File: mp257/v0.1/mp257-devboard.kicad_pcb (KiCad board)
At the start: 4 copper layers, 42.2 x 57.9 mm, 225 parts, among them CON1 microSDCon_SMT_104031-0811, J1 Pins_02x40_P0.4mm_W3.0mm_SMT, J2 Pins_02x40_P0.4mm_W3.0mm_SMT, J3 USB-C_Receptacle_Molex_217179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, J4 Pins_02x04_RightAngle_P2.54mm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, J5 Pins_01x02_RightAngle_P2.54mm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, J6 Pins_02x05_P1.27mm_SMT, J7 Conn_02x20_Odd_Even, U1 STM32MP257FAK3, U15 MT40A1G16TB-062E IT:F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

Commit message: Finish board, cleanup BOM
Parts:
- C225, C235: footprint 4ms_Capacitor:C_0201_TightCourtyard -> 4ms_Capacitor:C_0201
- J7: value Conn_02x20_Odd_Even -> Pins_02x20_P0.4mm_W3.0mm_SMT
- U9: value MCP1501-18xCH -> MCP1501T-18x/CHY
