File: mp257/v0.1/ddr.kicad_sch (KiCad schematic)
At the start: 63 parts, among them U1 STM32MP257FAK3, U15 MT40A1G16TB-062E IT:F

Commit message: mp257 placement WIP
Parts:
- C194: footprint 4ms_Capacitor:C_0603 -> 4ms_Capacitor:C_0402; symbol 4ms_Capacitor:10uF_0603_10V -> 4ms_Capacitor:10uF_0402_6.3V; Display 10uF/10V -> 10uF; Specifications 10uF, Min. 10V X5R 10% -> 10uF, Min. 6.3V, 0402, Ceramic/MLCC

Commit message: Mark: before re-doing RAM
Parts:
- removed C158, C221: 100nF_0402_16V, 4ms_Capacitor:C_0402, symbol 4ms_Capacitor:100nF_0402_16V

Commit message: All DDR nets length matched, and exported net report
Parts:
- R174: footprint 4ms_Resistor:R_0402 -> Resistor_SMD:R_0201_0603Metric; symbol 4ms_Resistor_0402:240Ω_0402 -> 4ms_Resistor_Misc:240Ω_0201; Specifications 240Ω, 1%, 1/16W, 0402 -> 240Ω, 5%, 0201
Changed lines of the file:
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@@
 	)
 	(symbol
-		(lib_id "4ms_Resistor_0402:240Ω_0402")
+		(lib_id "4ms_Resistor_Misc:240Ω_0201")
 		(at 125.73 168.91 0)
 		(unit 1)
@@
 			)
 		)
-		(property "Footprint" "4ms_Resistor:R_0402"
+		(property "Footprint" "Resistor_SMD:R_0201_0603Metric"
 			(at 123.19 181.864 0)
 			(effects
@@
 			)
 		)
-		(property "Description" "240Ω, 1%, 1/16W, 0402"
+		(property "Description" "240Ω, 5%, 0201"
 			(at 125.73 168.91 0)
 			(effects
@@
 			)
 		)
-		(property "Specifications" "240Ω, 1%, 1/16W, 0402"
+		(property "Specifications" "240Ω, 5%, 0201"
 			(at 123.19 176.53 0)
 			(effects

Commit message: Routing
Changed lines of the file:
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@@
 	(wire
 		(pts
-			(xy 367.03 90.17) (xy 369.57 90.17)
-		)
-		(stroke
-			(width 0)
-			(type default)
-		)
-	)
-	(wire
-		(pts
 			(xy 200.66 77.47) (xy 180.34 77.47)
 		)
@@
 	(wire
 		(pts
-			(xy 363.22 151.13) (xy 369.57 151.13)
-		)
-		(stroke
-			(width 0)
-			(type default)
-		)
-	)
-	(wire
-		(pts
 			(xy 54.61 87.63) (xy 31.75 87.63)
 		)
@@
 	(wire
 		(pts
-			(xy 364.49 130.81) (xy 369.57 130.81)
-		)
-		(stroke
-			(width 0)
-			(type default)
-		)
-	)
-	(wire
-		(pts
 			(xy 236.22 77.47) (xy 241.3 77.47)
 		)
@@
 		)
 	)
-	(label "VPP_DDR"
-		(at 241.3 184.15 0)
-		(effects
-			(font
-				(size 1.27 1.27)
-			)
-			(justify left bottom)
-		)
-	)
 	(label "DDR_A8"
 		(at 287.02 129.54 0)
@@
 			(effects
 				(font
+					(size 1.27 1.27)
+				)
+				(justify left)
+				(hide yes)
+			)
+		)
+	)
+	(global_label "VPP_DDR"
+		(shape input)
+		(at 241.3 184.15 0)
+		(fields_autoplaced yes)
+		(effects
+			(font
+				(size 1.27 1.27)
+			)
+			(justify left)
+		)
+		(property "Intersheetrefs" "${INTERSHEET_REFS}"
+			(at 252.6914 184.15 0)
+			(effects
+				(font

Commit message: Cleanup BOM, update all parts from lib
Parts:
- C194: value 10uF_0603_10V -> 10uF_0402_6.3V; JLCPCB ID C19702 -> (none); Manufacturer Murata -> (none); Part Number GRM188R61A106KE69D -> (none)
- R174: value 240Ω_0402 -> 240Ω_0201; JLCPCB ID C114755 -> (none); Manufacturer Yageo -> (none); Part Number RC0402FR-07240RL -> (none)
- U1: ALTIUM_VALUE STM32MP257FAK3 -> (none); COMPONENTLINK1URL http://tunmcdsvn.tun.st.com/Component_Documentation_Library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 -> (none); COMPONENT_COUNTRY_OF_ORIGIN Unknown -> (none); ID 5491 -> (none); INTERNAL_PART_NUMBER MCD-03375 -> (none); MANUFACTURER STMICROELECTRONICS -> (none); MANUFACTURER_PART_NUMBER STM32MP257FAK3 -> (none); Manufacturer (none) -> STMICROELECTRONICS; ORDER_CODE_DIGIKEY N/A -> (none); ORDER_CODE_FARNELL N/A -> (none); ORDER_CODE_RS N/A -> (none); PACKAGE TFBGA -> (none); PART_PREFERENCE Recommended -> (none); PART_TYPE IC -> (none); Part Number (none) -> STM32MP257FAK3; SHOWFIELDS YES -> (none); STATUS Checked -> (none); Specifications (none) -> STM32MP257FAK3 MPU
- U15: Manufacturer MICRON -> Winbond; Manufacturer 2 (none) -> ISSI; Manufacturer 3 (none) -> MICRON; Note (none) -> P/N 1 and 2 are 4Gb. P/N 3 is 16Gbit; Part Number MT40A1G16TB-062E IT:F -> W664GG6RB; Part Number 2 (none) -> IS43QR16256B-075UBLI; Part Number 3 (none) -> MT40A1G16TB-062E IT:F

Commit message: Missing p/n
Parts:
- C194: JLCPCB ID (none) -> C77000; Manufacturer (none) -> Murata; Part Number (none) -> GRM155R61A106ME44D
Changed lines of the file:
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@@
 			)
 		)
-		(property "Manufacturer" ""
+		(property "Manufacturer" "Murata"
 			(at 299.72 217.678 0)
 			(effects
@@
 			)
 		)
-		(property "Part Number" ""
+		(property "Part Number" "GRM155R61A106ME44D"
 			(at 299.72 219.202 0)
 			(effects
@@
 			)
 		)
-		(property "JLCPCB ID" ""
+		(property "JLCPCB ID" "C77000"
 			(at 303.53 220.98 0)
 			(effects
@@
 			(effects
 				(font
-					(size 1.27 1.27)
-				)
-				(hide yes)
-			)
-		)
-		(property "Note" ""
-			(at 302.26 208.28 0)
-			(effects
-				(font

Commit message: Missing p/n
Parts:
- R174: JLCPCB ID (none) -> C155745; Manufacturer (none) -> Yageo; Part Number (none) -> RC0201FR-07240RL
Changed lines of the file:
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@@
 			)
 		)
-		(property "Manufacturer" ""
+		(property "Manufacturer" "Yageo"
 			(at 123.19 178.308 0)
 			(effects
@@
 			)
 		)
-		(property "Part Number" ""
+		(property "Part Number" "RC0201FR-07240RL"
 			(at 123.19 180.086 0)
 			(effects
@@
 			)
 		)
-		(property "JLCPCB ID" ""
+		(property "JLCPCB ID" "C155745"
 			(at 123.19 183.642 0)
 			(effects
@@
 				(hide yes)
 			)
-		)
-		(property "Note" ""
-			(at 125.73 168.91 0)
-			(effects
-				(font
-					(size 1.27 1.27)
-				)
-				(hide yes)
-			)
