File: carrier-breakout/v0.2-ltdc/mp257-carrier-board.kicad_pcb (KiCad board)
At the start: 2 copper layers, 136.5 x 111.6 mm, 54 parts, among them J1 USB-C_Receptacle_Molex_217179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, J2 Eurorack_Power_10pin_Shrouded, J5 Conn_01x30_FPC_ER-TFT050-10, J6 Pins_02x40_P2.54mm_TH, J7 Pins_02x40_P2.54mm_TH, J9 Pins_02x40_P2.54mm_TH, U13 AP6230xZ6, U14 AP2411SN, U3 FUSB302BMPX, U6 TLV61046ADB

Commit message: mp257 carrier board mostly complete
Parts:
- removed C5: 47uF_5x5.3_16V, 4ms_Capacitor:CP_Elec_5x5.3
- removed C7: 100nF_0603_16V, 4ms_Capacitor:C_0603
- removed D3: B140HW-7, 4ms_Diode:D_SOD-123
- removed H1, H2, H3: Spacer Nylon, Unthreaded, Height=11mm, ID >= 3mm, OD < 6mm, 4ms_Hardware:MountingHole_Generic_3mm
- removed J9: Pins_02x40_P2.54mm_TH, 4ms_Connector:Pins_2x40_P2.54mm_TH
- added J11: Conn_02x15_Odd_Even, Connector_PinHeader_2.54mm:PinHeader_2x15_P2.54mm_Vertical, F.Cu at (0.00, 0.00)
- added J3: ~, 4ms_Connector_Card:mp153-devboard-sockets_A, F.Cu at (0.00, 0.00)
- added JP21, JP22: SolderJumper_2_Open, 4ms_SolderJumper:JUMPER_SMD_1x2_tiny, F.Cu at (0.00, 0.00)
Connections:
- J8 pad C10: unconnected-(J8-PI6-PadC10) -> /PI6
- J8 pad C12: unconnected-(J8-PI7-PadC12) -> /PI7
- J8 pad C13: unconnected-(J8-PG15-PadC13) -> /PG15
- J8 pad C14: unconnected-(J8-PG8-PadC14) -> /PG8
- J8 pad C15: unconnected-(J8-PI5-PadC15) -> /PI5
- J8 pad C16: unconnected-(J8-PG9-PadC16) -> /PG9
- J8 pad C17: unconnected-(J8-PI1-PadC17) -> /PI1
- J8 pad C18: unconnected-(J8-PG10-PadC18) -> /PG10
- J8 pad C19: unconnected-(J8-PI0-PadC19) -> /PI0
- J8 pad C20: unconnected-(J8-PG14-PadC20) -> /PG14
- J8 pad C21: unconnected-(J8-PI2-PadC21) -> /PI2
- J8 pad C22: unconnected-(J8-PG11-PadC22) -> /PG11
- J8 pad C23: unconnected-(J8-GND-PadC23) -> GND
- J8 pad C24: unconnected-(J8-PG13-PadC24) -> /PG13
- J8 pad C25: unconnected-(J8-GND-PadC25) -> GND
- J8 pad C26: unconnected-(J8-PF13-PadC26) -> /PF13
- J8 pad C27: unconnected-(J8-PG12-PadC27) -> /PG12
- J8 pad C28: unconnected-(J8-PF12-PadC28) -> /PF12
- J8 pad C29: unconnected-(J8-PI3-PadC29) -> /PI3
- J8 pad C30: unconnected-(J8-PF15-PadC30) -> /PF15
- J8 pad C31: unconnected-(J8-PI4-PadC31) -> /PI4
- J8 pad C32: unconnected-(J8-PF14-PadC32) -> /PF14
- J8 pad C33: unconnected-(J8-PH5-PadC33) -> /PH5
- J8 pad C34: unconnected-(J8-PG5-PadC34) -> /PG5
- J8 pad C35: unconnected-(J8-PH4-PadC35) -> /PH4
- J8 pad C36: unconnected-(J8-PG6-PadC36) -> /PG6
- J8 pad C37: unconnected-(J8-PF7-PadC37) -> /PF7
- J8 pad C38: unconnected-(J8-PI9-PadC38) -> /PI9
- J8 pad C39: unconnected-(J8-PF8-PadC39) -> /PF8
- J8 pad C40: unconnected-(J8-PG7-PadC40) -> /PG7
Routing:
- net GND: track 825.6 -> 1370.8 mm, vias 24 -> 26
- net +5V: track 192.2 -> 335.7 mm, vias 6 -> 7
- net +3V3: track 122.8 -> 252.4 mm, vias 1 -> 4
- net /USB_VBUS_JACK: track 103.6 -> 200.7 mm, vias 1 -> 4
- net /USB_JACK_D+: track 4.71 -> 91.0 mm, vias 1 -> 4
- net /USB_JACK_D-: track 5.24 -> 90.8 mm, vias 1 -> 2
- net /PI6: track 0.00 -> 80.9 mm
- net /PI7: track 0.00 -> 73.8 mm
- net /PG8: track 0.00 -> 70.2 mm
- net /PG9: track 0.00 -> 67.5 mm
- net /SCREEN_LED_ENABLE: track 0.00 -> 62.9 mm, vias 0 -> 2
- net /A57: track 49.2 -> 112.0 mm, vias 1 -> 2
- net /A63: track 58.6 -> 121.4 mm, vias 1 -> 2
- net /A61: track 53.3 -> 115.3 mm, vias 1 -> 0
- net /A59: track 51.1 -> 111.5 mm, vias 1 -> 0
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Other:
- board size 136.5 x 111.6 mm -> 136.5 x 169 mm
- board text added: "ADC"

Commit message: mp257 carrier board: finished and ordered with JLCPCB
Routing:
- net GND: track 1370.8 -> 1372.3 mm
- net /PF12: track 40.3 -> 39.2 mm
- net /PI7: track 73.8 -> 74.9 mm
- net /PI6: track 80.9 -> 81.9 mm
- net /PF15: track 36.2 -> 35.3 mm
- net /PF13: track 43.8 -> 42.9 mm
- net /PG10: track 58.1 -> 58.9 mm
- net /PF14: track 32.3 -> 31.5 mm
- net /PG8: track 70.2 -> 70.9 mm
- net /PG13: track 47.4 -> 46.8 mm
- net /PG9: track 67.5 -> 66.9 mm
- net /PG6: track 24.3 -> 23.7 mm
Other:
- board size 136.5 x 169 mm -> 123 x 166.2 mm
