File: carrier-breakout/v0.2-ltdc/mp257-carrier-board.kicad_sch (KiCad schematic)
At the start: 53 parts, among them J1 USB-C_Receptacle_Molex_217179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, J10 Conn_01x16, J2 Eurorack_Power_10pin_Shrouded, J5 Conn_01x30_FPC_ER-TFT050-10, J6 Pins_02x40_P2.54mm_TH, J7 Pins_02x40_P2.54mm_TH, J9 Conn_01x14, U13 AP6230xZ6, U14 AP2411SN, U3 FUSB302BMPX, U6 TLV61046ADB

Commit message: mp257 carrier board mostly complete
Parts:
- removed C5: 47uF_5x5.3_16V, 4ms_Capacitor:CP_Elec_5x5.3, symbol 4ms_Capacitor:47uF_5x5.3_16V
- removed C7: 100nF_0603_16V, 4ms_Capacitor:C_0603, symbol 4ms_Capacitor:100nF_0603_16V
- removed D3: B140HW-7, 4ms_Diode:D_SOD-123, symbol 4ms_Diode:B140HW-7
- removed J10: Conn_01x16, Connector_PinHeader_2.54mm:PinHeader_1x16_P2.54mm_Vertical, symbol Connector_Generic:Conn_01x16
- removed J9: Conn_01x14, Connector_PinHeader_2.54mm:PinHeader_1x14_P2.54mm_Vertical, symbol Connector_Generic:Conn_01x14
- added J11: Conn_02x15_Odd_Even, Connector_PinHeader_2.54mm:PinHeader_2x15_P2.54mm_Vertical, symbol Connector_Generic:Conn_02x15_Odd_Even
- added JP21, JP22: SolderJumper_2_Open, 4ms_SolderJumper:JUMPER_SMD_1x2_tiny, symbol 4ms_Net_Tie:SolderJumper_2_Open
- J8: footprint 4ms_Connector_Card:mp257-devboard-sockets_C -> 4ms_Connector_Card:mp153-devboard-sockets_C
Connections:
- net A1: now also JP21.2 (B)
- net A3: now also JP22.2 (B)
- net GND: now also J8.C23 (GND), J8.C25 (GND), J11.13 (Pin_13), J11.15 (Pin_15)
- net SCREEN_LED_ENABLE: now also JP21.1 (A)
- net SCREEN_RESET: now also JP22.1 (A)
- net PI6: now reaches J8.C10 (PI6)
- net PI6: now also J11.1 (Pin_1)
- net PI7: now reaches J8.C12 (PI7)
- net PI7: now also J11.2 (Pin_2)
- net PG15: now reaches J8.C13 (PG15)
- net PG15: now also J11.3 (Pin_3)
- net PG8: now reaches J8.C14 (PG8)
- net PG8: now also J11.4 (Pin_4)
- net PI5: now reaches J8.C15 (PI5)
- net PI5: now also J11.5 (Pin_5)
- net PG9: now reaches J8.C16 (PG9)
- net PG9: now also J11.6 (Pin_6)
- net PI1: now reaches J8.C17 (PI1)
- net PI1: now also J11.7 (Pin_7)
- net PG10: now reaches J8.C18 (PG10)
- net PG10: now also J11.8 (Pin_8)
- net PI0: now reaches J8.C19 (PI0)
- net PI0: now also J11.9 (Pin_9)
- net PG14: now reaches J8.C20 (PG14)
- net PG14: now also J11.10 (Pin_10)
- net PI2: now reaches J8.C21 (PI2)
- net PI2: now also J11.11 (Pin_11)
- net PG11: now reaches J8.C22 (PG11)
- net PG11: now also J11.12 (Pin_12)
- net PG13: now reaches J8.C24 (PG13)
- net PG13: now also J11.14 (Pin_14)
- net PF13: now reaches J8.C26 (PF13)
- net PF13: now also J11.16 (Pin_16)
- net PG12: now reaches J8.C27 (PG12)
- net PG12: now also J11.17 (Pin_17)
- net PF12: now reaches J8.C28 (PF12)
- net PF12: now also J11.18 (Pin_18)
- net PI3: now reaches J8.C29 (PI3)
- net PI3: now also J11.19 (Pin_19)
- net PF15: now reaches J8.C30 (PF15)
- net PF15: now also J11.20 (Pin_20)
- net PI4: now reaches J8.C31 (PI4)
- net PI4: now also J11.21 (Pin_21)
- net PF14: now reaches J8.C32 (PF14)
- net PF14: now also J11.22 (Pin_22)
- net PH5: now reaches J8.C33 (PH5)
- net PH5: now also J11.23 (Pin_23)
- net PG5: now reaches J8.C34 (PG5)
- net PG5: now also J11.24 (Pin_24)
- net PH4: now reaches J8.C35 (PH4)
- net PH4: now also J11.25 (Pin_25)
- net PG6: now reaches J8.C36 (PG6)
- net PG6: now also J11.26 (Pin_26)
- net PF7: now reaches J8.C37 (PF7)
- net PF7: now also J11.27 (Pin_27)
- net PI9: now reaches J8.C38 (PI9)
- net PI9: now also J11.28 (Pin_28)
- net PF8: now reaches J8.C39 (PF8)
- net PF8: now also J11.29 (Pin_29)
- net PG7: now reaches J8.C40 (PG7)
- net PG7: now also J11.30 (Pin_30)
Other:
- note added: "Breakout carrier board for mp257-devboard v0.1"
- note added: "Supports DRD (Host or Device mode). Will power attached USB Devices up to ~500mA. This circuit will not allow powering the board via the USB jack (to do that, an additional AP2411 is needed)"
- note removed: "Breakout carrier board for mp153-devboard v0.2"
- note removed: "Supports DRD (Host or Device mode). Will power attached USB Devices up to ~500mA. This circuit will not allow powering the mp153 board via the USB jack (to do that, an additional AP2411 is needed)"
- moved on the sheet: C11, C12, C3, C4, C6, C73, C74, D2, J2, L5, R35, R36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

Commit message: mp257 carrier board: finished and ordered with JLCPCB
Parts:
- J5: JLCPCB ID (none) -> C2856833
- U6: JLCPCB ID (none) -> C464815
